Commit message: feat: arm tuning for new joint

File: src/Arm/arm_srdf/config/arm_urdf.ros2_control.xacro (robot description, xacro)
@@ -32,5 +32,5 @@
         <param name="sensor_type">absolute</param> <!-- or "quadrature" -->
         <param name="sensor_ticks">4096</param>
-        <param name="sensor_offset">3.14</param>
+        <param name="sensor_offset">5.125</param>
         <param name="crossover">true</param> <!-- or "continuous" -->
         <param name="invert">false</param>
@@ -42,11 +42,11 @@
       <joint name="Joint_3">
         <param name="can_id">14</param>
-        <param name="kP">30.0</param>
+        <param name="kP">1.0</param>
         <param name="kI">0.0</param>
-        <param name="kD">3.0</param>
-        <param name="kF">125</param>
+        <param name="kD">0.0</param>
+        <param name="kF">60.0</param>
         <param name="sensor_type">absolute</param> <!-- or "quadrature" -->
         <param name="sensor_ticks">4096</param>
-        <param name="sensor_offset">2.85</param>
+        <param name="sensor_offset">3.35</param>
         <param name="crossover">true</param> <!-- or "continuous" -->
         <param name="invert">true</param>
@@ -64,5 +64,5 @@
         <param name="sensor_type">absolute</param> <!-- or "quadrature" -->
         <param name="sensor_ticks">4096</param>
-        <param name="sensor_offset">1.021</param>
+        <param name="sensor_offset">0.0</param>
         <param name="crossover">true</param> <!-- or "continuous" -->
         <param name="invert">false</param>
@@ -80,5 +80,5 @@
         <param name="sensor_type">absolute</param> <!-- or "quadrature" -->
         <param name="sensor_ticks">4096</param>
-        <param name="sensor_offset">2.48</param>
+        <param name="sensor_offset">6.05</param>
         <param name="crossover">true</param> <!-- or "continuous" -->
         <param name="invert">true</param>

File: src/Arm/arm_urdf/urdf/arm_urdf.urdf (robot description, URDF)
Before this commit: robot arm_urdf, 9 links, 8 joints
Joints:
- joint Joint_2: limit lower=-0.65 upper=0.2361743685324814 effort=100.0 velocity=0.10 -> lower=-0.694 upper=0.211 effort=100.0 velocity=0.10
- joint Joint_3: limit lower=-0.7417525505578109 upper=0.2139174802949436 effort=100.0 velocity=0.08 -> lower=-1.152 upper=1.80 effort=100.0 velocity=0.1

Commit message: tune: fix sensor offsets and limits

File: src/Arm/arm_srdf/config/arm_urdf.ros2_control.xacro (robot description, xacro)
@@ -32,5 +32,5 @@
         <param name="sensor_type">absolute</param> <!-- or "quadrature" -->
         <param name="sensor_ticks">4096</param>
-        <param name="sensor_offset">5.125</param>
+        <param name="sensor_offset">3.0</param>
         <param name="crossover">true</param> <!-- or "continuous" -->
         <param name="invert">false</param>
@@ -48,5 +48,5 @@
         <param name="sensor_type">absolute</param> <!-- or "quadrature" -->
         <param name="sensor_ticks">4096</param>
-        <param name="sensor_offset">3.35</param>
+        <param name="sensor_offset">-3.0</param>
         <param name="crossover">true</param> <!-- or "continuous" -->
         <param name="invert">true</param>
@@ -80,5 +80,5 @@
         <param name="sensor_type">absolute</param> <!-- or "quadrature" -->
         <param name="sensor_ticks">4096</param>
-        <param name="sensor_offset">6.05</param>
+        <param name="sensor_offset">0.4</param>
         <param name="crossover">true</param> <!-- or "continuous" -->
         <param name="invert">true</param>

File: src/Arm/arm_urdf/urdf/arm_urdf.urdf (robot description, URDF)
Before this commit: robot arm_urdf, 9 links, 8 joints
Joints:
- joint Joint_2: limit lower=-0.694 upper=0.211 effort=100.0 velocity=0.10 -> lower=-0.55 upper=0.31 effort=100.0 velocity=0.10
- joint Joint_3: limit lower=1.538 upper=2.402 effort=100.0 velocity=0.1 -> lower=-1.178 upper=0.957 effort=100.0 velocity=0.1
- joint Joint_5: limit lower=-1.371 upper=0.828 effort=100.0 velocity=1.0 -> lower=-1.7794 upper=0.655 effort=100.0 velocity=1.0

Commit message: Fix: wrong start up value when inverted

File: src/Arm/arm_srdf/config/arm_urdf.ros2_control.xacro (robot description, xacro)
@@ -34,5 +34,5 @@
         <param name="sensor_type">absolute</param> <!-- or "quadrature" -->
         <param name="sensor_ticks">4096</param>
-        <param name="sensor_offset">3.0</param>
+        <param name="sensor_offset">-2.7</param>
         <param name="crossover">true</param> <!-- or "continuous" -->
         <param name="invert">false</param>
@@ -51,5 +51,5 @@
         <param name="sensor_type">absolute</param> <!-- or "quadrature" -->
         <param name="sensor_ticks">4096</param>
-        <param name="sensor_offset">-3.0</param>
+        <param name="sensor_offset">3.14</param>
         <param name="crossover">true</param> <!-- or "continuous" -->
         <param name="invert">true</param>
@@ -68,5 +68,5 @@
         <param name="sensor_type">absolute</param> <!-- or "quadrature" -->
         <param name="sensor_ticks">4096</param>
-        <param name="sensor_offset">0.0</param>
+        <param name="sensor_offset">-1.0</param>
         <param name="crossover">true</param> <!-- or "continuous" -->
         <param name="invert">false</param>
@@ -85,5 +85,5 @@
         <param name="sensor_type">absolute</param> <!-- or "quadrature" -->
         <param name="sensor_ticks">4096</param>
-        <param name="sensor_offset">0.4</param>
+        <param name="sensor_offset">-0.23</param>
         <param name="crossover">true</param> <!-- or "continuous" -->
         <param name="invert">true</param>

File: src/Arm/arm_urdf/urdf/arm_urdf.urdf (robot description, URDF)
Before this commit: robot arm_urdf, 9 links, 8 joints
Joints:
- joint Joint_1: limit lower=-3.14 upper=3.14 effort=100.0 velocity=0.5 -> lower=-4.0 upper=4.0 effort=100.0 velocity=1.0
