Commit message: updating limits with encoder movement

File: src/Arm/arm_urdf/urdf/arm_urdf.urdf (robot description, URDF)
Before this commit: robot arm_urdf, 9 links, 8 joints
Joints:
- joint Joint_3: limit lower=-1.152 upper=1.80 effort=100.0 velocity=0.1 -> lower=1.538 upper=2.402 effort=100.0 velocity=0.1
- joint Joint_5: limit lower=-1.599417185 upper=1.1678841562 effort=100.0 velocity=1.0 -> lower=-1.371 upper=0.828 effort=100.0 velocity=1.0

Commit message: big guy

File: src/Arm/arm_urdf/urdf/arm_urdf.urdf (robot description, URDF)
Before this commit: robot arm_urdf, 9 links, 8 joints
Joints:
- joint Joint_3: limit lower=1.538 upper=2.402 effort=100.0 velocity=0.1 -> lower=-1.152 upper=1.80 effort=100.0 velocity=0.1

Commit message: URDF seems right

File: src/Arm/arm_urdf/urdf/arm_urdf.urdf (robot description, URDF)
Before this commit: robot arm_urdf, 9 links, 8 joints
Links:
- removed link Link_7
- removed link arm_base_link
- removed link eef_link
- added link EndEffector, mass 1.73621324847791; collision mesh filename=package://arm_urdf/meshes/EndEffector.STL; visual mesh filename=package://arm_urdf/meshes/EndEffector.STL
- link Link_1: mass 1.1012 -> 0.894465735151454; geometry collision mesh filename=package://arm_urdf/meshes/Link_1.STL; visual mesh filename=package://arm_urdf/meshes/Link_1.STL
- link Link_2: mass 0.73837 -> 1.06976490829179; geometry collision mesh filename=package://arm_urdf/meshes/Link_2.STL; visual mesh filename=package://arm_urdf/meshes/Link_2.STL
- link Link_3: mass 2.2244 -> 2.73505357681468; geometry collision mesh filename=package://arm_urdf/meshes/Link_3.STL; visual mesh filename=package://arm_urdf/meshes/Link_3.STL
- link Link_4: mass 0.72553 -> 0.592254181279744; geometry collision mesh filename=package://arm_urdf/meshes/Link_4.STL; visual mesh filename=package://arm_urdf/meshes/Link_4.STL
- link Link_5: mass 0.90226 -> 0.822677539380202; geometry collision mesh filename=package://arm_urdf/meshes/Link_5.STL; visual mesh filename=package://arm_urdf/meshes/Link_5.STL
- link Link_6: mass 0.496128874632715 -> 0.330260939704627; geometry collision mesh filename=package://arm_urdf/meshes/Link_6.STL; visual mesh filename=package://arm_urdf/meshes/Link_6.STL
Joints:
- removed joint arm_base_joint
- removed joint eef_joint
- joint Joint_1: origin xyz=0 0 0.022287 rpy=0 0 0 -> xyz=0 0 0.0287 rpy=0 0 0; type revolute -> continuous
- joint Joint_2: limit lower=-0.55 upper=0.31 effort=100.0 velocity=0.10 -> (none); origin xyz=-0.03175 0 0.1 rpy=0 0 0 -> xyz=0 0 0.10795 rpy=0 0 0; type revolute -> continuous
- joint Joint_3: axis 0 -1 0 -> 0 1 0; limit lower=-1.178 upper=0.957 effort=100.0 velocity=0.1 -> (none); origin xyz=0.4507 0 0.5371 rpy=0 0 0 -> xyz=0.068432 0 0.59125 rpy=0 0 0; type revolute -> continuous
- joint Joint_4: axis -0.99059 0 0.1369 -> 0 0 -1; limit lower=-3.14 upper=3.14 effort=100.0 velocity=0.5 -> (none); origin xyz=0.03191 0 -0.0044098 rpy=0 0 0 -> xyz=0 0.01165 0.077 rpy=0 0 0; type revolute -> continuous
- joint Joint_5: axis 0 -1 0 -> 0 1 0; limit lower=-1.7794 upper=0.655 effort=100.0 velocity=1.0 -> (none); origin xyz=0.68151 0 -0.094183 rpy=0 0 0 -> xyz=0 0 0.45756 rpy=0 0 0; type revolute -> continuous
- joint Joint_6: axis -1 0 0 -> 0 0 1; child Link_7 -> EndEffector; limit effort=100.0 velocity=1.0 -> (none); origin xyz=0.071675 -0.02785 0 rpy=0 0 0 -> xyz=0 -0.02785 0.022092 rpy=0 0 0
