Commit message: Collision via simple boxes

File: src/URDF/rover_urdf/urdf/arm_urdf.xacro (robot description, xacro)
@@ -33,11 +33,14 @@
         </visual>
         <collision>
-        <origin
-            xyz="0 0 0"
-            rpy="0 0 0" />
-        <geometry>
-            <mesh
-            filename="package://rover_urdf/meshes/Link_1.STL" />
-        </geometry>
+            <origin xyz="-0.028000 0.051000 -0.060000" rpy="0.000000 0.000000 0.000000"/>
+            <geometry>
+            <cylinder radius="0.020000" length="0.120000"/>
+            </geometry>
+        </collision>
+        <collision>
+            <origin xyz="0.000000 0.000000 0.014100" rpy="0.000000 0.000000 0.000000"/>
+            <geometry>
+            <box size="0.120000 0.212500 0.037300"/>
+            </geometry>
         </collision>
     </link>
@@ -73,11 +76,32 @@
         </visual>
         <collision>
-        <origin
-            xyz="0 0 0"
-            rpy="0 0 0" />
-        <geometry>
-            <mesh
-            filename="package://rover_urdf/meshes/Link_2.STL" />
-        </geometry>
+            <origin xyz="0.000000 -0.075000 0.110725" rpy="1.570000 0.000000 0.000000"/>
+            <geometry>
+            <cylinder radius="0.057833" length="0.122902"/>
+            </geometry>
+        </collision>
+        <collision>
+            <origin xyz="0.000000 0.059878 0.110725" rpy="1.570000 0.000000 0.000000"/>
+            <geometry>
+            <cylinder radius="0.057833" length="0.032902"/>
+            </geometry>
+        </collision>
+        <collision>
+            <origin xyz="0.000000 0.000000 0.000725" rpy="0.000000 0.000000 0.000000"/>
+            <geometry>
+            <box size="0.106750 0.104676 0.020363"/>
+            </geometry>
+        </collision>
+        <collision>
+            <origin xyz="0.000000 0.046000 0.040725" rpy="0.000000 0.000000 0.000000"/>
+            <geometry>
+            <box size="0.106750 0.014676 0.070363"/>
+            </geometry>
+        </collision>
+        <collision>
+            <origin xyz="0.000000 -0.046000 0.040725" rpy="0.000000 0.000000 0.000000"/>
+            <geometry>
+            <box size="0.106750 0.014676 0.070363"/>
+            </geometry>
         </collision>
     </link>
@@ -126,11 +150,62 @@
         </visual>
         <collision>
-        <origin
-            xyz="0 0 0"
-            rpy="0 0 0" />
-        <geometry>
-            <mesh
-            filename="package://rover_urdf/meshes/Link_3.STL" />
-        </geometry>
+            <origin xyz="0.070000 -0.034283 0.592000" rpy="1.570000 0.000000 0.000000"/>
+            <geometry>
+            <cylinder radius="0.050000" length="0.055272"/>
+            </geometry>
+        </collision>
+        <collision>
+            <origin xyz="0.070000 -0.094283 0.592000" rpy="1.570000 0.000000 0.000000"/>
+            <geometry>
+            <cylinder radius="0.015548" length="0.125272"/>
+            </geometry>
+        </collision>
+        <collision>
+            <origin xyz="0.070000 0.065717 0.592000" rpy="1.570000 0.000000 0.000000"/>
+            <geometry>
+            <cylinder radius="0.025548" length="0.045272"/>
+            </geometry>
+        </collision>
+        <collision>
+            <origin xyz="0.070000 0.040000 0.592000" rpy="1.570000 0.000000 0.000000"/>
+            <geometry>
+            <cylinder radius="0.045548" length="0.005272"/>
+            </geometry>
+        </collision>
+        <collision>
+            <origin xyz="0.020000 -0.015000 0.519808" rpy="0.000000 0.000000 0.000000"/>
+            <geometry>
+            <box size="0.048322 0.009363 0.148954"/>
+            </geometry>
+        </collision>
+        <collision>
+            <origin xyz="0.020000 0.039500 0.519808" rpy="0.000000 0.000000 0.000000"/>
+            <geometry>
+            <box size="0.048322 0.009363 0.148954"/>
+            </geometry>
+        </collision>
+        <collision>
+            <origin xyz="0.000000 0.012000 0.199808" rpy="0.000000 0.000000 0.000000"/>
+            <geometry>
+            <box size="0.048322 0.060000 0.488954"/>
+            </geometry>
+        </collision>
+        <collision>
+            <origin xyz="0.008289 0.045717 -0.000192" rpy="1.570000 0.000000 0.000000"/>
+            <geometry>
+            <cylinder radius="0.035548" length="0.020000"/>
+            </geometry>
+        </collision>
+        <collision>
+            <origin xyz="0.000000 -0.034283 0.199808" rpy="0.000000 0.000000 0.000000"/>
+            <geometry>
+            <box size="0.058322 0.029363 0.168954"/>
+            </geometry>
+        </collision>
+        <collision>
+            <origin xyz="-0.001711 0.055717 0.199808" rpy="0.000000 0.000000 0.000000"/>
+            <geometry>
+            <box size="0.078322 0.029363 0.238954"/>
+            </geometry>
         </collision>
     </link>
@@ -179,11 +254,20 @@
         </visual>
         <collision>
-        <origin
-            xyz="0 0 0"
-            rpy="0 0 0" />
-        <geometry>
-            <mesh
-            filename="package://rover_urdf/meshes/Link_4.STL" />
-        </geometry>
+            <origin xyz="0.000000 0.011650 0.024000" rpy="0.000000 0.000000 0.000000"/>
+            <geometry>
+            <box size="0.058549 0.030000 0.101500"/>
+            </geometry>
+        </collision>
+        <collision>
+            <origin xyz="-0.053000 0.011650 -0.016000" rpy="0.000000 0.000000 0.000000"/>
+            <geometry>
+            <cylinder radius="0.021000" length="0.145333"/>
+            </geometry>
+        </collision>
+        <collision>
+            <origin xyz="0.002098 0.011650 0.070000" rpy="0.000000 0.000000 0.000000"/>
+            <geometry>
+            <cylinder radius="0.038000" length="0.015333"/>
+            </geometry>
         </collision>
     </link>
@@ -232,11 +316,32 @@
         </visual>
         <collision>
-        <origin
-            xyz="0 0 0"
-            rpy="0 0 0" />
-        <geometry>
-            <mesh
-            filename="package://rover_urdf/meshes/Link_5.STL" />
-        </geometry>
+            <origin xyz="-0.000000 0.000000 0.211681" rpy="0.000000 0.000000 0.000000"/>
+            <geometry>
+            <cylinder radius="0.015267" length="0.397787"/>
+            </geometry>
+        </collision>
+        <collision>
+            <origin xyz="-0.000000 0.000000 0.001681" rpy="0.000000 0.000000 0.000000"/>
+            <geometry>
+            <cylinder radius="0.035267" length="0.007787"/>
+            </geometry>
+        </collision>
+        <collision>
+            <origin xyz="-0.000000 0.049800 0.458000" rpy="1.570000 0.000000 0.000000"/>
+            <geometry>
+            <cylinder radius="0.010100" length="0.107787"/>
+            </geometry>
+        </collision>
+        <collision>
+            <origin xyz="0.000000 0.019800 0.458000" rpy="1.570000 0.000000 0.000000"/>
+            <geometry>
+            <cylinder radius="0.045267" length="0.027787"/>
+            </geometry>
+        </collision>
+        <collision>
+            <origin xyz="-0.000000 -0.040200 0.451681" rpy="0.000000 0.000000 0.000000"/>
+            <geometry>
+            <box size="0.022900 0.008300 0.055841"/>
+            </geometry>
         </collision>
     </link>
@@ -285,11 +390,26 @@
         </visual>
         <collision>
-        <origin
-            xyz="0 0 0"
-            rpy="0 0 0" />
-        <geometry>
-            <mesh
-            filename="package://rover_urdf/meshes/Link_6.STL" />
-        </geometry>
+            <origin xyz="-0.017000 -0.069000 0.025888" rpy="0.000000 0.000000 0.000000"/>
+            <geometry>
+            <cylinder radius="0.011667" length="0.065592"/>
+            </geometry>
+        </collision>
+        <collision>
+            <origin xyz="-0.017000 -0.069000 0.063000" rpy="0.000000 0.000000 0.000000"/>
+            <geometry>
+            <cylinder radius="0.014000" length="0.009000"/>
+            </geometry>
+        </collision>
+        <collision>
+            <origin xyz="0.000000 -0.028000 0.030000" rpy="0.000000 0.000000 0.000000"/>
+            <geometry>
+            <box size="0.070000 0.015000 0.034194"/>
+            </geometry>
+        </collision>
+        <collision>
+            <origin xyz="0.000000 -0.028000 -0.000000" rpy="1.570000 0.000000 0.000000"/>
+            <geometry>
+            <cylinder radius="0.021667" length="0.015592"/>
+            </geometry>
         </collision>
     </link>
@@ -338,11 +458,26 @@
         </visual>
         <collision>
-        <origin
-            xyz="0 0 0"
-            rpy="0 0 0" />
-        <geometry>
-            <mesh
-            filename="package://rover_urdf/meshes/EndEffector.STL" />
-        </geometry>
+            <origin xyz="-0.000000 0.000000 0.270000" rpy="0.000000 0.000000 0.000000"/>
+            <geometry>
+            <box size="0.032381 0.240516 0.145815"/>
+            </geometry>
+        </collision>
+        <collision>
+            <origin xyz="0.000000 0.000000 0.202653" rpy="0.000000 0.000000 0.000000"/>
+            <geometry>
+            <box size="0.052381 0.240516 0.015815"/>
+            </geometry>
+        </collision>
+        <collision>
+            <origin xyz="-0.000000 0.000000 0.152653" rpy="0.000000 0.000000 0.000000"/>
+            <geometry>
+            <box size="0.062381 0.060516 0.095815"/>
+            </geometry>
+        </collision>
+        <collision>
+            <origin xyz="-0.000000 0.000000 0.070000" rpy="0.000000 0.000000 0.000000"/>
+            <geometry>
+            <cylinder radius="0.041587" length="0.051087"/>
+            </geometry>
         </collision>
     </link>

File: src/URDF/rover_urdf/urdf/chassis_urdf.xacro (robot description, xacro)
@@ -33,10 +33,55 @@
     </visual>
     <collision>
-      <origin
-        xyz="0 0 0"
-        rpy="0 0 0" />
-      <geometry>
-        <mesh
-          filename="package://rover_urdf/meshes/Frame.STL" />
+      <origin xyz="0.077212 0.000738 -0.070000" rpy="0.000000 0.000000 0.000000"/>
+      <geometry>
+        <box size="0.553312 0.472700 0.190000"/>
+      </geometry>
+    </collision>
+    <collision>
+      <origin xyz="-0.262788 0.078500 0.032719" rpy="0.000000 0.000000 0.000000"/>
+      <geometry>
+        <box size="0.153312 0.032700 0.277297"/>
+      </geometry>
+    </collision>
+    <collision>
+      <origin xyz="-0.180000 0.230000 0.000000" rpy="0.000000 0.000000 0.000000"/>
+      <geometry>
+        <box size="0.030000 0.030000 0.220000"/>
+      </geometry>
+    </collision>
+    <collision>
+      <origin xyz="-0.180000 -0.230000 0.000000" rpy="0.000000 0.000000 0.000000"/>
+      <geometry>
+        <box size="0.030000 0.030000 0.220000"/>
+      </geometry>
+    </collision>
+    <collision>
+      <origin xyz="0.360000 0.000000 0.000000" rpy="0.000000 0.000000 0.000000"/>
+      <geometry>
+        <box size="0.093312 0.072700 0.167297"/>
+      </geometry>
+    </collision>
+    <collision>
+      <origin xyz="0.360000 -0.140000 -0.050000" rpy="0.000000 0.000000 0.000000"/>
+      <geometry>
+        <box size="0.043312 0.072700 0.077297"/>
+      </geometry>
+    </collision>
+    <collision>
+      <origin xyz="0.360000 0.140000 -0.050000" rpy="0.000000 0.000000 0.000000"/>
+      <geometry>
+        <box size="0.043312 0.072700 0.077297"/>
+      </geometry>
+    </collision>
+    <collision>
+      <origin xyz="0.107212 0.180738 0.722719" rpy="0.000000 0.000000 0.000000"/>
+      <geometry>
+        <cylinder radius="0.021800" length="1.423063"/>
+      </geometry>
+    </collision>
+    <collision>
+      <origin xyz="0.105000 0.180738 1.445000" rpy="0.000000 0.000000 0.000000"/>
+      <geometry>
+        <box size="0.403312 0.042700 0.030000"/>
       </geometry>
     </collision>
@@ -73,10 +118,7 @@
     </visual>
     <collision>
-      <origin
-        xyz="0 0 0"
-        rpy="0 0 0" />
-      <geometry>
-        <mesh
-          filename="package://rover_urdf/meshes/Rocker_Right.STL" />
+      <origin xyz="0.000000 -0.041075 0.005650" rpy="0.000000 0.000000 0.000000"/>
+      <geometry>
+        <box size="0.150000 0.090000 0.240000"/>
       </geometry>
     </collision>
@@ -127,10 +169,13 @@
     </visual>
     <collision>
-      <origin
-        xyz="0 0 0"
-        rpy="0 0 0" />
-      <geometry>
-        <mesh
-          filename="package://rover_urdf/meshes/Sus_Arm_Front_Right.STL" />
+      <origin xyz="0.477000 -0.270000 0.084000" rpy="0.000000 0.000000 0.000000"/>
+      <geometry>
+        <box size="0.450000 0.090000 0.050000"/>
+      </geometry>
+    </collision>
+    <collision>
+      <origin xyz="0.624500 -0.345000 0.083000" rpy="0.000000 0.000000 0.000000"/>
+      <geometry>
+        <box size="0.085000 0.070000 0.090000"/>
       </geometry>
     </collision>
@@ -180,10 +225,19 @@
     </visual>
     <collision>
-      <origin
-        xyz="0 0 0"
-        rpy="0 0 0" />
-      <geometry>
-        <mesh
-          filename="package://rover_urdf/meshes/Wheel_Arm_Front_Right.STL" />
+      <origin xyz="-0.664057 -0.199347 -0.131243" rpy="0.000000 0.000000 0.000000"/>
+      <geometry>
+        <box size="0.154965 0.097667 0.148371"/>
+      </geometry>
+    </collision>
+    <collision>
+      <origin xyz="-0.664057 -0.125000 -0.051243" rpy="0.000000 0.000000 0.000000"/>
+      <geometry>
+        <box size="0.074965 0.049667 0.228371"/>
+      </geometry>
+    </collision>
+    <collision>
+      <origin xyz="-0.664057 -0.219347 0.045000" rpy="0.000000 0.000000 0.000000"/>
+      <geometry>
+        <box size="0.074965 0.157667 0.068371"/>
       </geometry>
     </collision>
@@ -233,10 +287,7 @@
     </visual>
     <collision>
-      <origin
-        xyz="0 0 0"
-        rpy="0 0 0" />
-      <geometry>
-        <mesh
-          filename="package://rover_urdf/meshes/Wheel_Front_Right.STL" />
+      <origin xyz="0.000000 -0.065254 0.000000" rpy="1.570000 0.000000 0.000000"/>
+      <geometry>
+        <cylinder radius="0.141667" length="0.139000"/>
       </geometry>
     </collision>
@@ -286,10 +337,13 @@
     </visual>
     <collision>
-      <origin
-        xyz="0 0 0"
-        rpy="0 0 0" />
-      <geometry>
-        <mesh
-          filename="package://rover_urdf/meshes/Sus_Arm_Back_Right.STL" />
+    <origin xyz="-0.477250 -0.271000 0.089000" rpy="0.000000 0.000000 0.000000"/>
+      <geometry>
+        <box size="0.451125 0.077375 0.060750"/>
+      </geometry>
+    </collision>
+    <collision>
+      <origin xyz="-0.627250 -0.347000 0.084000" rpy="0.000000 0.000000 0.000000"/>
+      <geometry>
+        <box size="0.081125 0.067375 0.090750"/>
       </geometry>
     </collision>
@@ -339,10 +393,19 @@
     </visual>
     <collision>
-      <origin
-        xyz="0 0 0"
-        rpy="0 0 0" />
-      <geometry>
-        <mesh
-          filename="package://rover_urdf/meshes/Wheel_Arm_Back_Right.STL" />
+      <origin xyz="-0.664057 -0.199347 -0.131243" rpy="0.000000 0.000000 0.000000"/>
+      <geometry>
+        <box size="0.154965 0.097667 0.148371"/>
+      </geometry>
+    </collision>
+    <collision>
+      <origin xyz="-0.664057 -0.125000 -0.051243" rpy="0.000000 0.000000 0.000000"/>
+      <geometry>
+        <box size="0.074965 0.049667 0.228371"/>
+      </geometry>
+    </collision>
+    <collision>
+      <origin xyz="-0.664057 -0.219347 0.045000" rpy="0.000000 0.000000 0.000000"/>
+      <geometry>
+        <box size="0.074965 0.157667 0.068371"/>
       </geometry>
     </collision>
@@ -392,10 +455,7 @@
     </visual>
     <collision>
-      <origin
-        xyz="0 0 0"
-        rpy="0 0 0" />
-      <geometry>
-        <mesh
-          filename="package://rover_urdf/meshes/Wheel_Back_Right.STL" />
+      <origin xyz="0.000000 -0.065254 0.000000" rpy="1.570000 0.000000 0.000000"/>
+      <geometry>
+        <cylinder radius="0.141667" length="0.139000"/>
       </geometry>
     </collision>
@@ -445,10 +505,7 @@
     </visual>
     <collision>
-      <origin
-        xyz="0 0 0"
-        rpy="0 0 0" />
-      <geometry>
-        <mesh
-          filename="package://rover_urdf/meshes/Rocker_Left.STL" />
+      <origin xyz="-0.000000 0.028855 0.005650" rpy="0.000000 0.000000 0.000000"/>
+      <geometry>
+        <box size="0.133500 0.090538 0.249925"/>
       </geometry>
     </collision>
@@ -499,10 +556,13 @@
     </visual>
     <collision>
-      <origin
-        xyz="0 0 0"
-        rpy="0 0 0" />
-      <geometry>
-        <mesh
-          filename="package://rover_urdf/meshes/Sus_Arm_Front_Left.STL" />
+      <origin xyz="0.477000 0.270000 0.084000" rpy="0.000000 0.000000 0.000000"/>
+      <geometry>
+        <box size="0.450000 0.090000 0.050000"/>
+      </geometry>
+    </collision>
+    <collision>
+      <origin xyz="0.624500 0.345000 0.083000" rpy="0.000000 0.000000 0.000000"/>
+      <geometry>
+        <box size="0.085000 0.070000 0.090000"/>
       </geometry>
     </collision>
@@ -552,10 +612,19 @@
     </visual>
     <collision>
-      <origin
-        xyz="0 0 0"
-        rpy="0 0 0" />
-      <geometry>
-        <mesh
-          filename="package://rover_urdf/meshes/Wheel_Arm_Front_Left.STL" />
+      <origin xyz="0.664057 0.199347 -0.131243" rpy="0.000000 0.000000 0.000000"/>
+      <geometry>
+        <box size="0.154965 0.097667 0.148371"/>
+      </geometry>
+    </collision>
+    <collision>
+      <origin xyz="0.664057 0.125000 -0.051243" rpy="0.000000 0.000000 0.000000"/>
+      <geometry>
+        <box size="0.074965 0.049667 0.228371"/>
+      </geometry>
+    </collision>
+    <collision>
+      <origin xyz="0.664057 0.219347 0.045000" rpy="0.000000 0.000000 0.000000"/>
+      <geometry>
+        <box size="0.074965 0.157667 0.068371"/>
       </geometry>
     </collision>
@@ -605,10 +674,7 @@
     </visual>
     <collision>
-      <origin
-        xyz="0 0 0"
-        rpy="0 0 0" />
-      <geometry>
-        <mesh
-          filename="package://rover_urdf/meshes/Wheel_Front_Left.STL" />
+      <origin xyz="0.000000 0.065254 0.000000" rpy="1.570000 0.000000 0.000000"/>
+      <geometry>
+        <cylinder radius="0.141667" length="0.139000"/>
       </geometry>
     </collision>
@@ -658,10 +724,13 @@
     </visual>
     <collision>
-      <origin
-        xyz="0 0 0"
-        rpy="0 0 0" />
-      <geometry>
-        <mesh
-          filename="package://rover_urdf/meshes/Sus_Arm_Back_Left.STL" />
+    <origin xyz="-0.477250 0.271000 0.089000" rpy="0.000000 0.000000 0.000000"/>
+      <geometry>
+        <box size="0.451125 0.077375 0.060750"/>
+      </geometry>
+    </collision>
+    <collision>
+      <origin xyz="-0.627250 0.347000 0.084000" rpy="0.000000 0.000000 0.000000"/>
+      <geometry>
+        <box size="0.081125 0.067375 0.090750"/>
       </geometry>
     </collision>
@@ -711,10 +780,19 @@
     </visual>
     <collision>
-      <origin
-        xyz="0 0 0"
-        rpy="0 0 0" />
-      <geometry>
-        <mesh
-          filename="package://rover_urdf/meshes/Wheel_Arm_Back_Left.STL" />
+      <origin xyz="0.664057 0.199347 -0.131243" rpy="0.000000 0.000000 0.000000"/>
+      <geometry>
+        <box size="0.154965 0.097667 0.148371"/>
+      </geometry>
+    </collision>
+    <collision>
+      <origin xyz="0.664057 0.125000 -0.051243" rpy="0.000000 0.000000 0.000000"/>
+      <geometry>
+        <box size="0.074965 0.049667 0.228371"/>
+      </geometry>
+    </collision>
+    <collision>
+      <origin xyz="0.664057 0.219347 0.045000" rpy="0.000000 0.000000 0.000000"/>
+      <geometry>
+        <box size="0.074965 0.157667 0.068371"/>
       </geometry>
     </collision>
@@ -764,10 +842,7 @@
     </visual>
     <collision>
-      <origin
-        xyz="0 0 0"
-        rpy="0 0 0" />
-      <geometry>
-        <mesh
-          filename="package://rover_urdf/meshes/Wheel_Back_Left.STL" />
+      <origin xyz="0.000000 0.065254 0.000000" rpy="1.570000 0.000000 0.000000"/>
+      <geometry>
+        <cylinder radius="0.141667" length="0.139000"/>
       </geometry>
     </collision>
@@ -817,10 +892,7 @@
     </visual>
     <collision>
-      <origin
-        xyz="0 0 0"
-        rpy="0 0 0" />
-      <geometry>
-        <mesh
-          filename="package://rover_urdf/meshes/Zed.STL" />
+      <origin xyz="0.028925 -0.008976 -0.010367" rpy="0.000000 0.290000 0.000000"/>
+      <geometry>
+        <box size="0.050000 0.183799 0.032000"/>
       </geometry>
     </collision>
@@ -870,10 +942,13 @@
     </visual>
     <collision>
-      <origin
-        xyz="0 0 0"
-        rpy="0 0 0" />
-      <geometry>
-        <mesh
-          filename="package://rover_urdf/meshes/GPS_Right.STL" />
+      <origin xyz="0.000000 0.000000 0.000000" rpy="0.000000 0.000000 0.000000"/>
+      <geometry>
+        <cylinder radius="0.080000" length="0.010000"/>
+      </geometry>
+    </collision>
+    <collision>
+      <origin xyz="0.000000 0.000000 0.013335" rpy="0.000000 0.000000 0.000000"/>
+      <geometry>
+        <box size="0.037470 0.037500 0.020000"/>
       </geometry>
     </collision>
@@ -923,10 +998,13 @@
     </visual>
     <collision>
-      <origin
-        xyz="0 0 0"
-        rpy="0 0 0" />
-      <geometry>
-        <mesh
-          filename="package://rover_urdf/meshes/GPS_Left.STL" />
+      <origin xyz="0.000000 0.000000 0.000000" rpy="0.000000 0.000000 0.000000"/>
+      <geometry>
+        <cylinder radius="0.080000" length="0.010000"/>
+      </geometry>
+    </collision>
+    <collision>
+      <origin xyz="0.000000 0.000000 0.013335" rpy="0.000000 0.000000 0.000000"/>
+      <geometry>
+        <box size="0.037470 0.037500 0.020000"/>
       </geometry>
     </collision>
@@ -976,10 +1054,7 @@
     </visual>
     <collision>
-      <origin
-        xyz="0 0 0"
-        rpy="0 0 0" />
-      <geometry>
-        <mesh
-          filename="package://rover_urdf/meshes/Antenna_Front.STL" />
+      <origin xyz="0.000042 -0.000128 0.150000" rpy="0.000000 0.000000 0.000000"/>
+      <geometry>
+        <cylinder radius="0.020000" length="0.300000"/>
       </geometry>
     </collision>
@@ -1029,10 +1104,7 @@
     </visual>
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