Commit message: feat: custom position vs trajectory mode

File: src/URDF/rover_urdf/urdf/arm_urdf.xacro (robot description, xacro)
@@ -108,5 +108,5 @@
     <joint
         name="Joint_1"
-        type="continuous">
+        type="revolute">
         <origin
         xyz="0 0 0.0287"
@@ -117,5 +117,6 @@
         link="Link_2" />
         <axis
-        xyz="0 0 1" />
+        xyz="0 0 -1" />
+        <limit lower="-3.3" upper="3.3" effort="100.0" velocity="0.1"/>
     </joint>
     <link
@@ -212,5 +213,5 @@
     <joint
         name="Joint_2"
-        type="continuous">
+        type="revolute">
         <origin
         xyz="0 0 0.10795"
@@ -222,4 +223,5 @@
         <axis
         xyz="0 -1 0" />
+        <limit lower="-3.14" upper="3.14" effort="100.0" velocity="0.2"/>
     </joint>
     <link
@@ -274,5 +276,5 @@
     <joint
         name="Joint_3"
-        type="continuous">
+        type="revolute">
         <origin
         xyz="0.068432 0 0.59125"
@@ -284,4 +286,5 @@
         <axis
         xyz="0 1 0" />
+        <limit lower="0" upper="2.84489" effort="100.0" velocity="0.2"/>
     </joint>
     <link
@@ -348,5 +351,5 @@
     <joint
         name="Joint_4"
-        type="continuous">
+        type="revolute">
         <origin
         xyz="0 0.01165 0.077"
@@ -358,4 +361,5 @@
         <axis
         xyz="0 0 -1" />
+        <limit lower="-3.14" upper="3.14" effort="100.0" velocity="0.2"/>
     </joint>
     <link
@@ -416,5 +420,5 @@
     <joint
         name="Joint_5"
-        type="continuous">
+        type="revolute">
         <origin
         xyz="0 0 0.45756"
@@ -425,5 +429,6 @@
         link="Link_6" />
         <axis
-        xyz="0 1 0" />
+        xyz="0 -1 0" />
+        <limit lower="-1.0" upper="1.0" effort="100.0" velocity="0.1"/>
     </joint>
     <link
@@ -494,4 +499,5 @@
         <axis
         xyz="0 0 1" />
+        <limit effort="100.0" velocity="0.3"/>
     </joint>
   </xacro:macro>
