Commit message: feat: switch moveit servo to joint trajectory controller

File: src/URDF/rover_urdf/urdf/arm_urdf.xacro (robot description, xacro)
@@ -343,5 +343,5 @@
         <axis
         xyz="0 0 -1" />
-        <limit lower="-3.14" upper="3.14" effort="100.0" velocity="1.2"/>
+        <limit lower="-3.14" upper="3.14" effort="100.0" velocity="0.5"/>
     </joint>
     <link
@@ -412,5 +412,5 @@
         <axis
         xyz="0 -1 0" />
-        <limit lower="-1.0" upper="1.0" effort="100.0" velocity="0.4"/>
+        <limit lower="-1.0" upper="1.0" effort="100.0" velocity="0.5"/>
     </joint>
     <link
@@ -481,5 +481,5 @@
         <axis
         xyz="0 0 1" />
-        <limit effort="100.0" velocity="0.8"/>
+        <limit effort="100.0" velocity="0.5"/>
     </joint>
   </xacro:macro>
