Commit message: feat: implement modeless teleop and move_group action server

File: src/URDF/rover_urdf/urdf/chassis_urdf.ros2_control.xacro (robot description, xacro)
@@ -38,7 +38,11 @@
       </joint>
       <joint name="Left_front_wheel_arm_joint">
+<<<<<<< HEAD
         <param name="node_id">2</param>
         <param name="multiplier">-0.0166666667</param>
         <param name="input_mode">Traj</param>
+=======
+        <param name="node_id">1</param>
+>>>>>>> cc5fb9f (feat: implement modeless teleop and move_group action server)
         <command_interface name="position"/>
         <state_interface name="position"/>
@@ -46,13 +50,21 @@
       <joint name="Left_back_wheel_arm_joint">
         <param name="node_id">3</param>
+<<<<<<< HEAD
         <param name="multiplier">0.0166666667</param>
         <param name="input_mode">Traj</param>
+=======
+>>>>>>> cc5fb9f (feat: implement modeless teleop and move_group action server)
         <command_interface name="position"/>
         <state_interface name="position"/>
       </joint>
       <joint name="Right_front_wheel_arm_joint">
+<<<<<<< HEAD
         <param name="node_id">1</param>
         <param name="input_mode">Traj</param>
         <param name="multiplier">0.0166666667</param>
+=======
+        <param name="node_id">2</param>
+        <param name="multiplier">1.0</param>
+>>>>>>> cc5fb9f (feat: implement modeless teleop and move_group action server)
         <command_interface name="position"/>
         <state_interface name="position"/>
@@ -60,6 +72,10 @@
       <joint name="Right_back_wheel_arm_joint">
         <param name="node_id">4</param>
+<<<<<<< HEAD
         <param name="input_mode">Traj</param>
         <param name="multiplier">-0.0166666667</param>
+=======
+        <param name="multiplier">1.0</param>
+>>>>>>> cc5fb9f (feat: implement modeless teleop and move_group action server)
         <command_interface name="position"/>
         <state_interface name="position"/>

File: src/URDF/rover_urdf/urdf/chassis_urdf.xacro (robot description, xacro)
@@ -802,5 +802,9 @@
     type="continuous">
     <origin
+<<<<<<< HEAD
       xyz="0 -0.01 0"
+=======
+      xyz="-.1 0 0"
+>>>>>>> cc5fb9f (feat: implement modeless teleop and move_group action server)
       rpy="0 0 0" />
     <parent

File: src/URDF/rover_urdf/urdf/rover_urdf.urdf.xacro (robot description, xacro)
@@ -31,3 +31,14 @@
     </joint>
   </xacro:if>
+<<<<<<< HEAD
+=======
+    <!-- Chassis ros2_control -->
+  <xacro:include filename="$(find rover_urdf)/urdf/chassis_urdf.ros2_control.xacro" />
+  <xacro:chassis_urdf_ros2_control name="ChassisSystem"/>
+  <joint name="base_link_to_chassis" type="fixed">
+    <parent link="base_link"/>
+    <child link="Frame"/>
+    <origin xyz="0 0 0" rpy="0 0 0"/>
+  </joint>
+>>>>>>> cc5fb9f (feat: implement modeless teleop and move_group action server)
 </robot>
