Commit message: end effector with placeholder values

File: src/URDF/rover_urdf/urdf/arm_urdf.ros2_control.xacro (robot description, xacro)
@@ -110,4 +110,21 @@
         <state_interface name="velocity"/>
       </joint>
+      <joint name="Joint_7"> <!-- for end effector -->
+        <param name="type">TalonSRX</param>
+        <param name="can_id">25</param> <!-- placeholder can_id -->
+        <param name="kP">0.012</param>
+        <param name="kI">0.0</param>
+        <param name="kD">0.0</param>
+        <param name="kF">0.005</param>
+        <param name="sensor_type">quadrature</param>
+        <param name="sensor_ticks">2163000</param> <!-- TODO: this number is close but not quite -->
+        <param name="sensor_offset">0.0</param>
+        <param name="crossover">true</param> <!-- or "continuous" -->
+        <param name="invert">true</param>
+        <param name="invert_sensor">true</param>
+        <command_interface name="position"/>
+        <state_interface name="position"/>
+        <state_interface name="velocity"/>
+      </joint>
     </ros2_control>
   </xacro:macro>

Commit message: 5/6 joints tuned

File: src/URDF/rover_urdf/urdf/arm_urdf.ros2_control.xacro (robot description, xacro)
@@ -5,36 +5,19 @@
       <hardware>
         <!-- By default, set up controllers for simulation. This won't work on real hardware -->
-        <plugin>mock_components/GenericSystem</plugin>
-        <!-- <plugin>ros2_control_rover_arm/RoverArmHardwareInterface</plugin> -->
+        <!-- <plugin>mock_components/GenericSystem</plugin> -->
+        <plugin>ros2_control_rover_arm/RoverArmHardwareInterface</plugin>
       </hardware>
       <joint name="Joint_1">
         <param name="type">TalonSRX</param>
-        <param name="can_id">10</param>
-        <param name="kP">3.0</param>
+        <param name="can_id">9</param>
+        <param name="kP">0.1</param>
         <param name="kI">0.0</param>
-        <param name="kD">1.0</param>
-        <param name="kF">0.5</param>
+        <param name="kD">0.0</param>
+        <param name="kF">0.0</param>
         <param name="sensor_type">absolute</param> <!-- or "quadrature" -->
         <param name="sensor_ticks">4096</param>
-        <param name="sensor_offset">0.0</param>
+        <param name="sensor_offset">1.0</param>
         <param name="crossover">true</param> <!-- or "continuous" -->
-        <param name="invert">false</param>
-        <param name="invert_sensor">true</param>
-        <command_interface name="position"/>
-        <state_interface name="position"/>
-        <state_interface name="velocity"/>
-      </joint>
-      <joint name="Joint_2">
-        <param name="type">TalonSRX</param>
-        <param name="can_id">11</param>
-        <param name="kP">10.0</param>
-        <param name="kI">0.0</param>
-        <param name="kD">10.0</param>
-        <param name="kF">100</param>
-        <param name="sensor_type">absolute</param> <!-- or "quadrature" -->
-        <param name="sensor_ticks">4096</param>
-        <param name="sensor_offset">-2.7</param>
-        <param name="crossover">true</param> <!-- or "continuous" -->
-        <param name="invert">false</param>
+        <param name="invert">true</param>
         <param name="invert_sensor">true</param>
         <command_interface name="position"/>
@@ -44,14 +27,14 @@
       <joint name="Joint_3">
         <param name="type">TalonSRX</param>
-        <param name="can_id">14</param>
-        <param name="kP">1.0</param>
-        <param name="kI">0.0</param>
+        <param name="can_id">11</param>
+        <param name="kP">60.0</param>
+        <param name="kI">1.0</param>
         <param name="kD">0.0</param>
-        <param name="kF">60.0</param>
+        <param name="kF">0.0</param>
         <param name="sensor_type">absolute</param> <!-- or "quadrature" -->
         <param name="sensor_ticks">4096</param>
-        <param name="sensor_offset">3.14</param>
-        <param name="crossover">true</param> <!-- or "continuous" -->
-        <param name="invert">true</param>
+        <param name="sensor_offset">-1.25</param>
+        <param name="crossover">false</param> <!-- or "continuous" -->
+        <param name="invert">false</param>
         <param name="invert_sensor">false</param>
         <command_interface name="position"/>
@@ -61,12 +44,29 @@
       <joint name="Joint_4">
         <param name="type">TalonSRX</param>
-        <param name="can_id">15</param>
-        <param name="kP">2.0</param>
+        <param name="can_id">12</param>
+        <param name="kP">1.0</param>
         <param name="kI">0.0</param>
         <param name="kD">0.0</param>
-        <param name="kF">5.0</param>
+        <param name="kF">0.0</param>
         <param name="sensor_type">absolute</param> <!-- or "quadrature" -->
         <param name="sensor_ticks">4096</param>
-        <param name="sensor_offset">-1.0</param>
+        <param name="sensor_offset">1.57</param>
+        <param name="crossover">true</param> <!-- or "continuous" -->
+        <param name="invert">true</param>
+        <param name="invert_sensor">true</param>
+        <command_interface name="position"/>
+        <state_interface name="position"/>
+        <state_interface name="velocity"/>
+      </joint>
+      <joint name="Joint_5">
+        <param name="type">TalonSRX</param>
+        <param name="can_id">19</param>
+        <param name="kP">100.0</param>
+        <param name="kI">0.0</param>
+        <param name="kD">0.0</param>
+        <param name="kF">0.0</param>
+        <param name="sensor_type">absolute</param> <!-- or "quadrature" -->
+        <param name="sensor_ticks">4096</param>
+        <param name="sensor_offset">5.25</param>
         <param name="crossover">true</param> <!-- or "continuous" -->
         <param name="invert">false</param>
@@ -76,30 +76,34 @@
         <state_interface name="velocity"/>
       </joint>
-      <joint name="Joint_5">
-        <param name="type">TalonSRX</param>
-        <param name="can_id">12</param>
-        <param name="kP">20.0</param>
-        <param name="kI">0.0</param>
-        <param name="kD">0.0</param>
-        <param name="kF">7.8</param>
-        <param name="sensor_type">absolute</param> <!-- or "quadrature" -->
-        <param name="sensor_ticks">4096</param>
-        <param name="sensor_offset">-0.23</param>
-        <param name="crossover">true</param> <!-- or "continuous" -->
-        <param name="invert">true</param>
-        <param name="invert_sensor">true</param>
+    </ros2_control>
+    <ros2_control name="${name}_odrive" type="system">
+      <hardware>
+        <!-- By default, set up controllers for simulation. This won't work on real hardware -->
+        <!-- <plugin>mock_components/GenericSystem</plugin> -->
+        <plugin>odrive_ros2_control_plugin/ODriveHardwareInterface</plugin>
+        <param name="can">can0</param>
+      </hardware>
+      <joint name="Joint_2">
+        <param name="node_id">10</param>
+        <param name="multiplier">-1.0</param>
         <command_interface name="position"/>
         <state_interface name="position"/>
         <state_interface name="velocity"/>
       </joint>
+    </ros2_control>
+    <ros2_control name="${name}_fake" type="system">
+      <hardware>
+        <!-- By default, set up controllers for simulation. This won't work on real hardware -->
+        <plugin>mock_components/GenericSystem</plugin>
+      </hardware>
       <joint name="Joint_6">
         <param name="type">TalonSRX</param>
         <param name="can_id">13</param>
-        <param name="kP">0.012</param>
+        <param name="kP">1.0</param>
         <param name="kI">0.0</param>
         <param name="kD">0.0</param>
-        <param name="kF">0.005</param>
-        <param name="sensor_type">quadrature</param> <!-- or "quadrature" -->
-        <param name="sensor_ticks">2163000</param> <!-- TODO: this number is close but not quite -->
+        <param name="kF">0.0</param>
+        <param name="sensor_type">absolute</param> <!-- or "quadrature" -->
+        <param name="sensor_ticks">4096</param> <!-- TODO: this number is close but not quite -->
         <param name="sensor_offset">0.0</param>
         <param name="crossover">true</param> <!-- or "continuous" -->

File: src/URDF/rover_urdf/urdf/arm_urdf.xacro (robot description, xacro)
@@ -108,5 +108,5 @@
     <joint
         name="Joint_1"
-        type="continuous">
+        type="revolute">
         <origin
         xyz="0 0 0.0287"
@@ -118,4 +118,5 @@
         <axis
         xyz="0 0 1" />
+        <limit lower="-3.2" upper="3.2" effort="100.0" velocity="0.2"/>
     </joint>
     <link
@@ -212,5 +213,5 @@
     <joint
         name="Joint_2"
-        type="continuous">
+        type="revolute">
         <origin
         xyz="0 0 0.10795"
@@ -222,4 +223,5 @@
         <axis
         xyz="0 -1 0" />
+        <limit lower="-3.14" upper="3.14" effort="100.0" velocity="0.2"/>
     </joint>
     <link
@@ -274,5 +276,5 @@
     <joint
         name="Joint_3"
-        type="continuous">
+        type="revolute">
         <origin
         xyz="0.068432 0 0.59125"
@@ -284,4 +286,5 @@
         <axis
         xyz="0 1 0" />
+        <limit lower="0" upper="2.84489" effort="100.0" velocity="0.2"/>
     </joint>
     <link
@@ -348,5 +351,5 @@
     <joint
         name="Joint_4"
-        type="continuous">
+        type="revolute">
         <origin
         xyz="0 0.01165 0.077"
@@ -358,4 +361,5 @@
         <axis
         xyz="0 0 -1" />
+        <limit lower="-3.14" upper="3.14" effort="100.0" velocity="0.2"/>
     </joint>
     <link
@@ -416,5 +420,5 @@
     <joint
         name="Joint_5"
-        type="continuous">
+        type="revolute">
         <origin
         xyz="0 0 0.45756"
@@ -425,5 +429,6 @@
         link="Link_6" />
         <axis
-        xyz="0 1 0" />
+        xyz="0 -1 0" />
+        <limit lower="-1.0" upper="1.0" effort="100.0" velocity="0.3"/>
     </joint>
     <link

Commit message: end effector launch and phoenix

File: src/URDF/rover_urdf/urdf/arm_urdf.ros2_control.xacro (robot description, xacro)
@@ -110,21 +110,4 @@
         <state_interface name="velocity"/>
       </joint>
-      <joint name="Joint_7"> <!-- for end effector -->
-        <param name="type">TalonSRX</param>
-        <param name="can_id">25</param> <!-- placeholder can_id -->
-        <param name="kP">0.012</param>
-        <param name="kI">0.0</param>
-        <param name="kD">0.0</param>
-        <param name="kF">0.005</param>
-        <param name="sensor_type">quadrature</param>
-        <param name="sensor_ticks">2163000</param> <!-- TODO: this number is close but not quite -->
-        <param name="sensor_offset">0.0</param>
-        <param name="crossover">true</param> <!-- or "continuous" -->
-        <param name="invert">true</param>
-        <param name="invert_sensor">true</param>
-        <command_interface name="position"/>
-        <state_interface name="position"/>
-        <state_interface name="velocity"/>
-      </joint>
     </ros2_control>
   </xacro:macro>

Commit message: Last joint working (ish)

File: src/URDF/rover_urdf/urdf/arm_urdf.ros2_control.xacro (robot description, xacro)
@@ -17,5 +17,5 @@
         <param name="sensor_type">absolute</param> <!-- or "quadrature" -->
         <param name="sensor_ticks">4096</param>
-        <param name="sensor_offset">1.0</param>
+        <param name="sensor_offset">4.1</param>
         <param name="crossover">true</param> <!-- or "continuous" -->
         <param name="invert">true</param>
@@ -76,4 +76,21 @@
         <state_interface name="velocity"/>
       </joint>
+      <joint name="Joint_6">
+        <param name="type">TalonSRX</param>
+        <param name="can_id">20</param>
+        <param name="kP">0.1</param>
+        <param name="kI">0.0</param>
+        <param name="kD">0.0</param>
+        <param name="kF">0.0</param>
+        <param name="sensor_type">absolute</param> <!-- or "quadrature" -->
+        <param name="sensor_ticks">4096</param> <!-- TODO: this number is close but not quite -->
+        <param name="sensor_offset">0.0</param>
+        <param name="crossover">true</param> <!-- or "continuous" -->
+        <param name="invert">false</param>
+        <param name="invert_sensor">true</param>
+        <command_interface name="position"/>
+        <state_interface name="position"/>
+        <state_interface name="velocity"/>
+      </joint>
     </ros2_control>
     <ros2_control name="${name}_odrive" type="system">
@@ -92,27 +109,4 @@
       </joint>
     </ros2_control>
-    <ros2_control name="${name}_fake" type="system">
-      <hardware>
-        <!-- By default, set up controllers for simulation. This won't work on real hardware -->
-        <plugin>mock_components/GenericSystem</plugin>
-      </hardware>
-      <joint name="Joint_6">
-        <param name="type">TalonSRX</param>
-        <param name="can_id">13</param>
-        <param name="kP">1.0</param>
-        <param name="kI">0.0</param>
-        <param name="kD">0.0</param>
-        <param name="kF">0.0</param>
-        <param name="sensor_type">absolute</param> <!-- or "quadrature" -->
-        <param name="sensor_ticks">4096</param> <!-- TODO: this number is close but not quite -->
-        <param name="sensor_offset">0.0</param>
-        <param name="crossover">true</param> <!-- or "continuous" -->
-        <param name="invert">true</param>
-        <param name="invert_sensor">true</param>
-        <command_interface name="position"/>
-        <state_interface name="position"/>
-        <state_interface name="velocity"/>
-      </joint>
-    </ros2_control>
   </xacro:macro>
 </robot>

File: src/URDF/rover_urdf/urdf/arm_urdf.xacro (robot description, xacro)
@@ -118,5 +118,5 @@
         <axis
         xyz="0 0 1" />
-        <limit lower="-3.2" upper="3.2" effort="100.0" velocity="0.2"/>
+        <limit lower="-3.3" upper="3.3" effort="100.0" velocity="0.2"/>
     </joint>
     <link

Commit message: WIP

File: src/URDF/rover_urdf/urdf/arm_urdf.ros2_control.xacro (robot description, xacro)
@@ -76,21 +76,4 @@
         <state_interface name="velocity"/>
       </joint>
-      <joint name="Joint_6">
-        <param name="type">TalonSRX</param>
-        <param name="can_id">20</param>
-        <param name="kP">0.1</param>
-        <param name="kI">0.0</param>
-        <param name="kD">0.0</param>
-        <param name="kF">0.0</param>
-        <param name="sensor_type">absolute</param> <!-- or "quadrature" -->
-        <param name="sensor_ticks">4096</param> <!-- TODO: this number is close but not quite -->
-        <param name="sensor_offset">0.0</param>
-        <param name="crossover">true</param> <!-- or "continuous" -->
-        <param name="invert">false</param>
-        <param name="invert_sensor">true</param>
-        <command_interface name="position"/>
-        <state_interface name="position"/>
-        <state_interface name="velocity"/>
-      </joint>
     </ros2_control>
     <ros2_control name="${name}_odrive" type="system">
@@ -109,4 +92,27 @@
       </joint>
     </ros2_control>
+    <ros2_control name="${name}" type="system">
+      <hardware>
+        <!-- By default, set up controllers for simulation. This won't work on real hardware -->
+        <plugin>mock_components/GenericSystem</plugin>
+      </hardware>
+      <joint name="Joint_6">
+        <param name="type">TalonSRX</param>
+        <param name="can_id">20</param>
+        <param name="kP">5.0</param>
+        <param name="kI">0.0</param>
+        <param name="kD">0.0</param>
+        <param name="kF">0.0</param>
+        <param name="sensor_type">absolute</param> <!-- or "quadrature" -->
+        <param name="sensor_ticks">4096</param> <!-- TODO: this number is close but not quite -->
+        <param name="sensor_offset">0.0</param>
+        <param name="crossover">true</param> <!-- or "continuous" -->
+        <param name="invert">false</param>
+        <param name="invert_sensor">true</param>
+        <command_interface name="position"/>
+        <state_interface name="position"/>
+        <state_interface name="velocity"/>
+      </joint>
+    </ros2_control>
   </xacro:macro>
 </robot>

Commit message: WIP

File: src/URDF/rover_urdf/urdf/arm_urdf.ros2_control.xacro (robot description, xacro)
@@ -17,5 +17,5 @@
         <param name="sensor_type">absolute</param> <!-- or "quadrature" -->
         <param name="sensor_ticks">4096</param>
-        <param name="sensor_offset">4.1</param>
+        <param name="sensor_offset">3.14</param>
         <param name="crossover">true</param> <!-- or "continuous" -->
         <param name="invert">true</param>
@@ -76,4 +76,21 @@
         <state_interface name="velocity"/>
       </joint>
+      <joint name="Joint_6">
+        <param name="type">TalonSRX</param>
+        <param name="can_id">20</param>
+        <param name="kP">1.0</param>
+        <param name="kI">0.0</param>
+        <param name="kD">0.0</param>
+        <param name="kF">0.0</param>
+        <param name="sensor_type">absolute</param> <!-- or "quadrature" -->
+        <param name="sensor_ticks">4096</param>
+        <param name="sensor_offset">0.0</param>
+        <param name="crossover">true</param> <!-- or "continuous" -->
+        <param name="invert">false</param>
+        <param name="invert_sensor">false</param>
+        <command_interface name="position"/>
+        <state_interface name="position"/>
+        <state_interface name="velocity"/>
+      </joint>
     </ros2_control>
     <ros2_control name="${name}_odrive" type="system">
@@ -92,26 +109,9 @@
       </joint>
     </ros2_control>
-    <ros2_control name="${name}" type="system">
+    <ros2_control name="${name}_fake" type="system">
       <hardware>
         <!-- By default, set up controllers for simulation. This won't work on real hardware -->
         <plugin>mock_components/GenericSystem</plugin>
       </hardware>
-      <joint name="Joint_6">
-        <param name="type">TalonSRX</param>
-        <param name="can_id">20</param>
-        <param name="kP">5.0</param>
-        <param name="kI">0.0</param>
-        <param name="kD">0.0</param>
-        <param name="kF">0.0</param>
-        <param name="sensor_type">absolute</param> <!-- or "quadrature" -->
-        <param name="sensor_ticks">4096</param> <!-- TODO: this number is close but not quite -->
-        <param name="sensor_offset">0.0</param>
-        <param name="crossover">true</param> <!-- or "continuous" -->
-        <param name="invert">false</param>
-        <param name="invert_sensor">true</param>
-        <command_interface name="position"/>
-        <state_interface name="position"/>
-        <state_interface name="velocity"/>
-      </joint>
     </ros2_control>
   </xacro:macro>

File: src/URDF/rover_urdf/urdf/arm_urdf.xacro (robot description, xacro)
@@ -430,5 +430,5 @@
         <axis
         xyz="0 -1 0" />
-        <limit lower="-1.0" upper="1.0" effort="100.0" velocity="0.3"/>
+        <limit lower="-1.0" upper="1.0" effort="100.0" velocity="0.1"/>
     </joint>
     <link
@@ -499,4 +499,5 @@
         <axis
         xyz="0 0 1" />
+        <limit effort="100.0" velocity="0.3"/>
     </joint>
   </xacro:macro>

Commit message: Arm changes efore mission control

File: src/URDF/rover_urdf/urdf/arm_urdf.ros2_control.xacro (robot description, xacro)
@@ -10,5 +10,5 @@
       <joint name="Joint_1">
         <param name="type">TalonSRX</param>
-        <param name="can_id">9</param>
+        <param name="can_id">14</param>
         <param name="kP">0.1</param>
         <param name="kI">0.0</param>
@@ -17,5 +17,5 @@
         <param name="sensor_type">absolute</param> <!-- or "quadrature" -->
         <param name="sensor_ticks">4096</param>
-        <param name="sensor_offset">3.14</param>
+        <param name="sensor_offset">4.14</param>
         <param name="crossover">true</param> <!-- or "continuous" -->
         <param name="invert">true</param>
@@ -34,5 +34,5 @@
         <param name="sensor_type">absolute</param> <!-- or "quadrature" -->
         <param name="sensor_ticks">4096</param>
-        <param name="sensor_offset">-1.25</param>
+        <param name="sensor_offset">0.0</param> <!-- -1.25 -->
         <param name="crossover">false</param> <!-- or "continuous" -->
         <param name="invert">false</param>
@@ -68,5 +68,5 @@
         <param name="sensor_type">absolute</param> <!-- or "quadrature" -->
         <param name="sensor_ticks">4096</param>
-        <param name="sensor_offset">5.25</param>
+        <param name="sensor_offset">4.0</param>
         <param name="crossover">true</param> <!-- or "continuous" -->
         <param name="invert">false</param>
@@ -78,5 +78,5 @@
       <joint name="Joint_6">
         <param name="type">TalonSRX</param>
-        <param name="can_id">20</param>
+        <param name="can_id">15</param>
         <param name="kP">1.0</param>
         <param name="kI">0.0</param>
@@ -84,7 +84,7 @@
         <param name="kF">0.0</param>
         <param name="sensor_type">absolute</param> <!-- or "quadrature" -->
-        <param name="sensor_ticks">4096</param>
+        <param name="sensor_ticks">1000</param>
         <param name="sensor_offset">0.0</param>
-        <param name="crossover">true</param> <!-- or "continuous" -->
+        <param name="continuous">true</param> <!-- or "crossover" -->
         <param name="invert">false</param>
         <param name="invert_sensor">false</param>

File: src/URDF/rover_urdf/urdf/arm_urdf.xacro (robot description, xacro)
@@ -118,5 +118,5 @@
         <axis
         xyz="0 0 1" />
-        <limit lower="-3.3" upper="3.3" effort="100.0" velocity="0.2"/>
+        <limit lower="-3.3" upper="3.3" effort="100.0" velocity="0.1"/>
     </joint>
     <link
