Commit message: feat: arm urdf and tuning

File: src/URDF/rover_urdf/urdf/arm_urdf.ros2_control.xacro (robot description, xacro)
@@ -5,37 +5,20 @@
       <hardware>
         <!-- By default, set up controllers for simulation. This won't work on real hardware -->
-        <plugin>mock_components/GenericSystem</plugin>
-        <!-- <plugin>ros2_control_rover_arm/RoverArmHardwareInterface</plugin> -->
+        <!-- <plugin>mock_components/GenericSystem</plugin> -->
+        <plugin>ros2_control_rover_arm/RoverArmHardwareInterface</plugin>
       </hardware>
       <joint name="Joint_1">
         <param name="type">TalonSRX</param>
-        <param name="can_id">10</param>
-        <param name="kP">3.0</param>
+        <param name="can_id">14</param>
+        <param name="kP">5.0</param>
         <param name="kI">0.0</param>
         <param name="kD">1.0</param>
-        <param name="kF">0.5</param>
+        <param name="kF">0.0</param>
         <param name="sensor_type">absolute</param> <!-- or "quadrature" -->
         <param name="sensor_ticks">4096</param>
-        <param name="sensor_offset">0.0</param>
+        <param name="sensor_offset">1.57</param>
         <param name="crossover">true</param> <!-- or "continuous" -->
         <param name="invert">false</param>
-        <param name="invert_sensor">true</param>
-        <command_interface name="position"/>
-        <state_interface name="position"/>
-        <state_interface name="velocity"/>
-      </joint>
-      <joint name="Joint_2">
-        <param name="type">TalonSRX</param>
-        <param name="can_id">11</param>
-        <param name="kP">10.0</param>
-        <param name="kI">0.0</param>
-        <param name="kD">10.0</param>
-        <param name="kF">100</param>
-        <param name="sensor_type">absolute</param> <!-- or "quadrature" -->
-        <param name="sensor_ticks">4096</param>
-        <param name="sensor_offset">-2.7</param>
-        <param name="crossover">true</param> <!-- or "continuous" -->
-        <param name="invert">false</param>
-        <param name="invert_sensor">true</param>
+        <param name="invert_sensor">false</param>
         <command_interface name="position"/>
         <state_interface name="position"/>
@@ -44,14 +27,14 @@
       <joint name="Joint_3">
         <param name="type">TalonSRX</param>
-        <param name="can_id">14</param>
-        <param name="kP">1.0</param>
-        <param name="kI">0.0</param>
-        <param name="kD">0.0</param>
-        <param name="kF">60.0</param>
+        <param name="can_id">11</param>
+        <param name="kP">4.0</param>
+        <param name="kI">0.1</param>
+        <param name="kD">0.5</param>
+        <param name="kF">0.0</param>
         <param name="sensor_type">absolute</param> <!-- or "quadrature" -->
         <param name="sensor_ticks">4096</param>
-        <param name="sensor_offset">3.14</param>
+        <param name="sensor_offset">-1.29154</param>
         <param name="crossover">true</param> <!-- or "continuous" -->
-        <param name="invert">true</param>
+        <param name="invert">false</param>
         <param name="invert_sensor">false</param>
         <command_interface name="position"/>
@@ -61,12 +44,29 @@
       <joint name="Joint_4">
         <param name="type">TalonSRX</param>
-        <param name="can_id">15</param>
-        <param name="kP">2.0</param>
+        <param name="can_id">12</param>
+        <param name="kP">1.0</param>
         <param name="kI">0.0</param>
         <param name="kD">0.0</param>
-        <param name="kF">5.0</param>
+        <param name="kF">0.0</param>
         <param name="sensor_type">absolute</param> <!-- or "quadrature" -->
         <param name="sensor_ticks">4096</param>
-        <param name="sensor_offset">-1.0</param>
+        <param name="sensor_offset">1.6057</param>
+        <param name="crossover">true</param> <!-- or "continuous" -->
+        <param name="invert">true</param>
+        <param name="invert_sensor">true</param>
+        <command_interface name="position"/>
+        <state_interface name="position"/>
+        <state_interface name="velocity"/>
+      </joint>
+      <joint name="Joint_5">
+        <param name="type">TalonSRX</param>
+        <param name="can_id">19</param>
+        <param name="kP">2.0</param>
+        <param name="kI">0.1</param>
+        <param name="kD">0.2</param>
+        <param name="kF">0.0</param>
+        <param name="sensor_type">absolute</param> <!-- or "quadrature" -->
+        <param name="sensor_ticks">4096</param>
+        <param name="sensor_offset">0.191986</param>
         <param name="crossover">true</param> <!-- or "continuous" -->
         <param name="invert">false</param>
@@ -76,32 +76,15 @@
         <state_interface name="velocity"/>
       </joint>
-      <joint name="Joint_5">
+      <joint name="Joint_6">
         <param name="type">TalonSRX</param>
-        <param name="can_id">12</param>
-        <param name="kP">20.0</param>
+        <param name="can_id">15</param>
+        <param name="kP">0.15</param>
         <param name="kI">0.0</param>
         <param name="kD">0.0</param>
-        <param name="kF">7.8</param>
-        <param name="sensor_type">absolute</param> <!-- or "quadrature" -->
-        <param name="sensor_ticks">4096</param>
-        <param name="sensor_offset">-0.23</param>
-        <param name="crossover">true</param> <!-- or "continuous" -->
-        <param name="invert">true</param>
-        <param name="invert_sensor">true</param>
-        <command_interface name="position"/>
-        <state_interface name="position"/>
-        <state_interface name="velocity"/>
-      </joint>
-      <joint name="Joint_6">
-        <param name="type">TalonSRX</param>
-        <param name="can_id">13</param>
-        <param name="kP">0.012</param>
-        <param name="kI">0.0</param>
-        <param name="kD">0.0</param>
-        <param name="kF">0.005</param>
+        <param name="kF">0.0</param>
         <param name="sensor_type">quadrature</param> <!-- or "quadrature" -->
-        <param name="sensor_ticks">2163000</param> <!-- TODO: this number is close but not quite -->
+        <param name="sensor_ticks">2039808</param>
         <param name="sensor_offset">0.0</param>
-        <param name="crossover">true</param> <!-- or "continuous" -->
+        <param name="continuous">true</param> <!-- or "crossover" -->
         <param name="invert">true</param>
         <param name="invert_sensor">true</param>
@@ -111,4 +94,25 @@
       </joint>
     </ros2_control>
+    <ros2_control name="${name}_odrive" type="system">
+      <hardware>
+        <!-- By default, set up controllers for simulation. This won't work on real hardware -->
+        <!-- <plugin>mock_components/GenericSystem</plugin> -->
+        <plugin>odrive_ros2_control_plugin/ODriveHardwareInterface</plugin>
+        <param name="can">can0</param>
+      </hardware>
+      <joint name="Joint_2">
+        <param name="node_id">10</param>
+        <param name="multiplier">-1.0</param>
+        <command_interface name="position"/>
+        <state_interface name="position"/>
+        <state_interface name="velocity"/>
+      </joint>
+    </ros2_control>
+    <ros2_control name="${name}_fake" type="system">
+      <hardware>
+        <!-- By default, set up controllers for simulation. This won't work on real hardware -->
+        <plugin>mock_components/GenericSystem</plugin>
+      </hardware>
+    </ros2_control>
   </xacro:macro>
 </robot>

Commit message: feat: arm tuning

File: src/URDF/rover_urdf/urdf/arm_urdf.ros2_control.xacro (robot description, xacro)
@@ -11,6 +11,6 @@
         <param name="type">TalonSRX</param>
         <param name="can_id">14</param>
-        <param name="kP">5.0</param>
-        <param name="kI">0.0</param>
+        <param name="kP">11.0</param>
+        <param name="kI">0.0005</param>
         <param name="kD">1.0</param>
         <param name="kF">0.0</param>
@@ -18,5 +18,5 @@
         <param name="sensor_ticks">4096</param>
         <param name="sensor_offset">1.57</param>
-        <param name="crossover">true</param> <!-- or "continuous" -->
+        <param name="crossover">false</param> <!-- or "continuous" -->
         <param name="invert">false</param>
         <param name="invert_sensor">false</param>
@@ -28,12 +28,12 @@
         <param name="type">TalonSRX</param>
         <param name="can_id">11</param>
-        <param name="kP">4.0</param>
-        <param name="kI">0.1</param>
-        <param name="kD">0.5</param>
+        <param name="kP">6.0</param>
+        <param name="kI">0.001</param>
+        <param name="kD">0.01</param>
         <param name="kF">0.0</param>
         <param name="sensor_type">absolute</param> <!-- or "quadrature" -->
         <param name="sensor_ticks">4096</param>
         <param name="sensor_offset">-1.29154</param>
-        <param name="crossover">true</param> <!-- or "continuous" -->
+        <param name="crossover">false</param> <!-- or "continuous" -->
         <param name="invert">false</param>
         <param name="invert_sensor">false</param>
@@ -45,6 +45,6 @@
         <param name="type">TalonSRX</param>
         <param name="can_id">12</param>
-        <param name="kP">1.0</param>
-        <param name="kI">0.0</param>
+        <param name="kP">4.0</param>
+        <param name="kI">0.001</param>
         <param name="kD">0.0</param>
         <param name="kF">0.0</param>
@@ -52,5 +52,5 @@
         <param name="sensor_ticks">4096</param>
         <param name="sensor_offset">1.6057</param>
-        <param name="crossover">true</param> <!-- or "continuous" -->
+        <param name="crossover">false</param> <!-- or "continuous" -->
         <param name="invert">true</param>
         <param name="invert_sensor">true</param>
@@ -62,12 +62,12 @@
         <param name="type">TalonSRX</param>
         <param name="can_id">19</param>
-        <param name="kP">2.0</param>
-        <param name="kI">0.1</param>
-        <param name="kD">0.2</param>
+        <param name="kP">8.5</param>
+        <param name="kI">0.001</param>
+        <param name="kD">0.001</param>
         <param name="kF">0.0</param>
         <param name="sensor_type">absolute</param> <!-- or "quadrature" -->
         <param name="sensor_ticks">4096</param>
         <param name="sensor_offset">0.191986</param>
-        <param name="crossover">true</param> <!-- or "continuous" -->
+        <param name="crossover">false</param> <!-- or "continuous" -->
         <param name="invert">false</param>
         <param name="invert_sensor">false</param>
@@ -79,6 +79,6 @@
         <param name="type">TalonSRX</param>
         <param name="can_id">15</param>
-        <param name="kP">0.15</param>
-        <param name="kI">0.0</param>
+        <param name="kP">0.01</param>
+        <param name="kI">0.000001</param>
         <param name="kD">0.0</param>
         <param name="kF">0.0</param>

File: src/URDF/rover_urdf/urdf/arm_urdf.xacro (robot description, xacro)
@@ -118,5 +118,5 @@
         <axis
         xyz="0 0 -1" />
-        <limit lower="-3.3" upper="3.3" effort="100.0" velocity="0.1"/>
+        <limit lower="-6.3" upper="6.3" effort="100.0" velocity="0.5"/>
     </joint>
     <link
@@ -361,5 +361,5 @@
         <axis
         xyz="0 0 -1" />
-        <limit lower="-3.14" upper="3.14" effort="100.0" velocity="0.2"/>
+        <limit lower="-3.14" upper="3.14" effort="100.0" velocity="0.8"/>
     </joint>
     <link
@@ -430,5 +430,5 @@
         <axis
         xyz="0 -1 0" />
-        <limit lower="-1.0" upper="1.0" effort="100.0" velocity="0.1"/>
+        <limit lower="-1.0" upper="1.0" effort="100.0" velocity="0.4"/>
     </joint>
     <link
@@ -499,5 +499,5 @@
         <axis
         xyz="0 0 1" />
-        <limit effort="100.0" velocity="0.3"/>
+        <limit effort="100.0" velocity="0.6"/>
     </joint>
   </xacro:macro>

Commit message: feat: updated URDF + CAN IDs

File: src/URDF/rover_urdf/urdf/arm_urdf.ros2_control.xacro (robot description, xacro)
@@ -7,8 +7,9 @@
         <!-- <plugin>mock_components/GenericSystem</plugin> -->
         <plugin>ros2_control_rover_arm/RoverArmHardwareInterface</plugin>
+        <param name="rw_rate">200</param>
       </hardware>
       <joint name="Joint_1">
         <param name="type">TalonSRX</param>
-        <param name="can_id">14</param>
+        <param name="can_id">9</param>
         <param name="kP">11.0</param>
         <param name="kI">0.0005</param>
@@ -18,5 +19,5 @@
         <param name="load_sensor">absolute</param>
         <param name="sensor_ticks">4096</param>
-        <param name="sensor_offset">4.99</param>
+        <param name="sensor_offset">4.88</param>
         <param name="crossover">false</param> <!-- or "continuous" -->
         <param name="invert">false</param>
@@ -29,19 +30,19 @@
         <param name="type">TalonSRX</param>
         <param name="can_id">11</param>
-        <param name="kP">14.0</param>
-        <param name="kI">0.0005</param>
-        <param name="kD">0.3</param>
+        <param name="kP">11.0</param>
+        <param name="kI">0.0</param>
+        <param name="kD">0.0</param>
         <param name="kF">0.0</param>
         <param name="sensor_type">quadrature</param>
         <param name="load_sensor">absolute</param>
         <param name="sensor_ticks">4096</param>
-        <param name="sensor_offset">1.9</param>
+        <param name="sensor_offset">-1.2</param>
         <param name="crossover">false</param> <!-- or "continuous" -->
         <param name="invert">false</param>
+        <param name="debug_frequency">1</param>
+        <param name="invert_sensor">false</param>
         <param name="gravity_ff_freq">10</param>
         <param name="current_frame">Link_4</param>
-        <param name="gravity_const">-0.03</param>
-        <param name="debug_frequency">1</param>
-        <param name="invert_sensor">false</param>
+        <param name="gravity_const">-0.023</param>
         <command_interface name="position"/>
         <state_interface name="position"/>
@@ -51,5 +52,5 @@
         <param name="type">TalonSRX</param>
         <param name="can_id">12</param>
-        <param name="kP">4.0</param>
+        <param name="kP">6.0</param>
         <param name="kI">0.001</param>
         <param name="kD">0.0</param>
@@ -58,5 +59,5 @@
         <param name="load_sensor">absolute</param>
         <param name="sensor_ticks">4096</param>
-        <param name="sensor_offset">4.69494</param>
+        <param name="sensor_offset">3.5</param>
         <param name="crossover">false</param> <!-- or "continuous" -->
         <param name="invert">true</param>
@@ -66,26 +67,8 @@
         <state_interface name="velocity"/>
       </joint>
-      <joint name="Joint_5">
-        <param name="type">TalonSRX</param>
-        <param name="can_id">19</param>
-        <param name="kP">8.5</param>
-        <param name="kI">0.001</param>
-        <param name="kD">0.001</param>
-        <param name="kF">0.0</param>
-        <param name="sensor_type">quadrature</param>
-        <param name="load_sensor">absolute</param>
-        <param name="sensor_ticks">4096</param>
-        <param name="sensor_offset">3.26377</param>
-        <param name="crossover">false</param> <!-- or "continuous" -->
-        <param name="invert">false</param>
-        <param name="invert_sensor">false</param>
-        <command_interface name="position"/>
-        <state_interface name="position"/>
-        <state_interface name="velocity"/>
-      </joint>
       <joint name="Joint_6">
         <param name="type">TalonSRX</param>
-        <param name="can_id">15</param>
-        <param name="kP">0.01</param>
+        <param name="can_id">14</param>
+        <param name="kP">0.015</param>
         <param name="kI">0.000001</param>
         <param name="kD">0.0</param>
@@ -112,4 +95,14 @@
         <param name="node_id">10</param>
         <param name="multiplier">-1.0</param>
+        <param name="gravity_ff_freq">30</param>
+        <param name="current_frame">Link_3</param>
+        <param name="gravity_const">-0.035</param>
+        <command_interface name="position"/>
+        <state_interface name="position"/>
+        <state_interface name="velocity"/>
+      </joint>
+      <joint name="Joint_5">
+        <param name="node_id">13</param>
+        <param name="multiplier">1.0</param>
         <command_interface name="position"/>
         <state_interface name="position"/>

File: src/URDF/rover_urdf/urdf/arm_urdf.xacro (robot description, xacro)
@@ -118,5 +118,5 @@
         <axis
         xyz="0 0 -1" />
-        <limit lower="-6.3" upper="6.3" effort="100.0" velocity="0.5"/>
+        <limit lower="-3.2" upper="5.5" effort="100.0" velocity="0.5"/>
     </joint>
     <link
@@ -151,5 +151,5 @@
         </visual>
         <collision>
-            <origin xyz="0.070000 -0.034283 0.592000" rpy="1.570000 0.000000 0.000000"/>
+            <origin xyz="-0.008 -0.034283 0.5" rpy="1.570000 0.000000 0.000000"/>
             <geometry>
             <cylinder radius="0.050000" length="0.055272"/>
@@ -157,5 +157,5 @@
         </collision>
         <collision>
-            <origin xyz="0.070000 -0.094283 0.592000" rpy="1.570000 0.000000 0.000000"/>
+            <origin xyz="-0.008 -0.094283 0.50" rpy="1.570000 0.000000 0.000000"/>
             <geometry>
             <cylinder radius="0.015548" length="0.125272"/>
@@ -163,5 +163,5 @@
         </collision>
         <collision>
-            <origin xyz="0.070000 0.065717 0.592000" rpy="1.570000 0.000000 0.000000"/>
+            <origin xyz="-0.008 0.065717 0.50" rpy="1.570000 0.000000 0.000000"/>
             <geometry>
             <cylinder radius="0.025548" length="0.045272"/>
@@ -169,19 +169,7 @@
         </collision>
         <collision>
-            <origin xyz="0.070000 0.040000 0.592000" rpy="1.570000 0.000000 0.000000"/>
+            <origin xyz="-0.008 0.040000 0.50" rpy="1.570000 0.000000 0.000000"/>
             <geometry>
             <cylinder radius="0.045548" length="0.005272"/>
-            </geometry>
-        </collision>
-        <collision>
-            <origin xyz="0.020000 -0.015000 0.519808" rpy="0.000000 0.000000 0.000000"/>
-            <geometry>
-            <box size="0.048322 0.009363 0.148954"/>
-            </geometry>
-        </collision>
-        <collision>
-            <origin xyz="0.020000 0.039500 0.519808" rpy="0.000000 0.000000 0.000000"/>
-            <geometry>
-            <box size="0.048322 0.009363 0.148954"/>
             </geometry>
         </collision>
@@ -223,5 +211,5 @@
         <axis
         xyz="0 -1 0" />
-        <limit lower="-3.14" upper="3.14" effort="100.0" velocity="0.2"/>
+        <limit lower="-3.14" upper="3.14" effort="100.0" velocity="0.5"/>
     </joint>
     <link
@@ -278,5 +266,5 @@
         type="revolute">
         <origin
-        xyz="0.068432 0 0.59125"
+        xyz="-0.0084125 0 0.50011"
         rpy="0 0 0" />
         <parent
@@ -286,5 +274,5 @@
         <axis
         xyz="0 1 0" />
-        <limit lower="0" upper="2.84489" effort="100.0" velocity="0.2"/>
+        <limit lower="0" upper="1.968" effort="100.0" velocity="0.4"/>
     </joint>
     <link
@@ -321,5 +309,5 @@
             <origin xyz="-0.000000 0.000000 0.211681" rpy="0.000000 0.000000 0.000000"/>
             <geometry>
-            <cylinder radius="0.015267" length="0.397787"/>
+            <cylinder radius="0.015267" length="0.24"/>
             </geometry>
         </collision>
@@ -331,17 +319,11 @@
         </collision>
         <collision>
-            <origin xyz="-0.000000 0.049800 0.458000" rpy="1.570000 0.000000 0.000000"/>
-            <geometry>
-            <cylinder radius="0.010100" length="0.107787"/>
-            </geometry>
-        </collision>
-        <collision>
-            <origin xyz="0.000000 0.019800 0.458000" rpy="1.570000 0.000000 0.000000"/>
-            <geometry>
-            <cylinder radius="0.045267" length="0.027787"/>
-            </geometry>
-        </collision>
-        <collision>
-            <origin xyz="-0.000000 -0.040200 0.451681" rpy="0.000000 0.000000 0.000000"/>
+            <origin xyz="-0.000000 0.049800 0.288" rpy="1.570000 0.000000 0.000000"/>
+            <geometry>
+            <cylinder radius="0.02" length="0.08"/>
+            </geometry>
+        </collision>
+        <collision>
+            <origin xyz="-0.000000 -0.040200 0.271681" rpy="0.000000 0.000000 0.000000"/>
             <geometry>
             <box size="0.022900 0.008300 0.055841"/>
@@ -353,5 +335,5 @@
         type="revolute">
         <origin
-        xyz="0 0.01165 0.077"
+        xyz="0 0.014035 0.062"
         rpy="0 0 0" />
         <parent
@@ -361,5 +343,5 @@
         <axis
         xyz="0 0 -1" />
-        <limit lower="-3.14" upper="3.14" effort="100.0" velocity="0.8"/>
+        <limit lower="-3.14" upper="3.14" effort="100.0" velocity="1.2"/>
     </joint>
     <link
@@ -394,5 +376,5 @@
         </visual>
         <collision>
-            <origin xyz="-0.017000 -0.069000 0.025888" rpy="0.000000 0.000000 0.000000"/>
+            <origin xyz="-0.02 -0.069000 -0.004" rpy="0.000000 0.000000 0.000000"/>
             <geometry>
             <cylinder radius="0.011667" length="0.065592"/>
@@ -400,5 +382,5 @@
         </collision>
         <collision>
-            <origin xyz="-0.017000 -0.069000 0.063000" rpy="0.000000 0.000000 0.000000"/>
+            <origin xyz="-0.02 -0.069000 0.033112" rpy="0.000000 0.000000 0.000000"/>
             <geometry>
             <cylinder radius="0.014000" length="0.009000"/>
@@ -422,5 +404,5 @@
         type="revolute">
         <origin
-        xyz="0 0 0.45756"
+        xyz="0 0 0.28676"
         rpy="0 0 0" />
         <parent
@@ -491,5 +473,5 @@
         type="continuous">
         <origin
-        xyz="0 -0.02785 0.022092"
+        xyz="0 -0.02585 0.031336"
         rpy="0 0 0" />
         <parent
