Commit message: fix: some arm tuning

File: src/URDF/rover_urdf/urdf/arm_urdf.ros2_control.xacro (robot description, xacro)
@@ -7,5 +7,5 @@
         <!-- <plugin>mock_components/GenericSystem</plugin> -->
         <plugin>ros2_control_rover_arm/RoverArmHardwareInterface</plugin>
-        <param name="rw_rate">200</param>
+        <param name="rw_rate">100</param>
       </hardware>
       <joint name="Joint_1">
@@ -19,5 +19,5 @@
         <param name="load_sensor">absolute</param>
         <param name="sensor_ticks">4096</param>
-        <param name="sensor_offset"> 0.997</param>
+        <param name="sensor_offset"> 2.6767</param>
         <param name="crossover">false</param> <!-- or "continuous" -->
         <param name="invert">false</param>
@@ -73,7 +73,7 @@
         <param name="type">TalonSRX</param>
         <param name="can_id">14</param>
-        <param name="kP">0.015</param>
+        <param name="kP">0.02</param>
         <param name="kI">0.000001</param>
-        <param name="kD">0.0</param>
+        <param name="kD">0.001</param>
         <param name="kF">0.0</param>
         <param name="sensor_type">quadrature</param> <!-- or "quadrature" -->

File: src/URDF/rover_urdf/urdf/arm_urdf.xacro (robot description, xacro)
@@ -481,5 +481,5 @@
         <axis
         xyz="0 0 1" />
-        <limit effort="100.0" velocity="0.6"/>
+        <limit effort="100.0" velocity="0.8"/>
     </joint>
   </xacro:macro>
