Commit message: visual looks good

File: src/URDF/rover_urdf/urdf/chassis_urdf.xacro (robot description, xacro)
@@ -143,5 +143,5 @@
       <origin
         xyz="0.57785416680796 -0.285312653930359 0.0825439600785206"
-        rpy="0 0 0" />
+        rpy="0 0 3.14" />
       <mass
         value="1.30155339210532" />
@@ -157,8 +157,8 @@
       <origin
         xyz="0 0 0"
-        rpy="0 0 0" />
-      <geometry>
-        <mesh
-          filename="package://rover_urdf/meshes/Sus_Arm_Front_Right.STL" />
+        rpy="0 0 3.14" />
+      <geometry>
+        <mesh
+          filename="package://rover_urdf/meshes/Sus_Arm_LB_RF.STL" />
       </geometry>
       <material
@@ -185,5 +185,5 @@
     type="fixed">
     <origin
-      xyz="-0.225 0.20619 -0.09"
+      xyz="0.43 -0.05 0"
       rpy="0 0 0" />
     <parent
@@ -199,5 +199,5 @@
       <origin
         xyz="-0.664037126098315 -0.188170529908974 -0.095574626273163"
-        rpy="0 0 0" />
+        rpy="0 0 3.14" />
       <mass
         value="1.37511463184065" />
@@ -213,8 +213,8 @@
       <origin
         xyz="0 0 0"
-        rpy="0 0 0" />
-      <geometry>
-        <mesh
-          filename="package://rover_urdf/meshes/Wheel_Arm_Front_Right.STL" />
+        rpy="0 0 3.14" />
+      <geometry>
+        <mesh
+          filename="package://rover_urdf/meshes/Wheel_Arm.STL" />
       </geometry>
       <material
@@ -245,7 +245,7 @@
   <joint
     name="Right_front_wheel_arm_joint"
-    type="fixed">
-    <origin
-      xyz="1.328 0.00105 0"
+    type="continuous">
+    <origin
+      xyz= "0 0 0"
       rpy="0 0 0" />
     <parent
@@ -254,5 +254,5 @@
       link="Wheel_Arm_Front_Right" />
     <axis
-      xyz="0 0 0" />
+      xyz="0 0 1" />
   </joint>
   <link
@@ -278,5 +278,5 @@
       <geometry>
         <mesh
-          filename="package://rover_urdf/meshes/Wheel_Right.STL" />
+          filename="package://rover_urdf/meshes/Wheel.STL" />
       </geometry>
       <material
@@ -297,5 +297,5 @@
     type="continuous">
     <origin
-      xyz="-0.664 -0.20693 -0.128"
+      xyz="0 0 -0.15"
       rpy="0 0 0" />
     <parent
@@ -328,5 +328,5 @@
       <geometry>
         <mesh
-          filename="package://rover_urdf/meshes/Sus_Arm_Back_Right.STL" />
+          filename="package://rover_urdf/meshes/Sus_Arm_LF_RB.STL" />
       </geometry>
       <material
@@ -353,5 +353,5 @@
     type="fixed">
     <origin
-      xyz="0.225 0.20619 -0.09"
+      xyz="-0.43 -0.05 0"
       rpy="0 0 0" />
     <parent
@@ -367,5 +367,5 @@
       <origin
         xyz="-0.664037126098314 -0.178170529908975 -0.0955746262731632"
-        rpy="0 0 0" />
+        rpy="0 0 3.14" />
       <mass
         value="1.37511463184065" />
@@ -381,8 +381,8 @@
       <origin
         xyz="0 0 0"
-        rpy="0 0 0" />
-      <geometry>
-        <mesh
-          filename="package://rover_urdf/meshes/Wheel_Arm_Back_Right.STL" />
+        rpy="0 0 3.14" />
+      <geometry>
+        <mesh
+          filename="package://rover_urdf/meshes/Wheel_Arm.STL" />
       </geometry>
       <material
@@ -413,5 +413,5 @@
   <joint
     name="Right_back_wheel_arm_joint"
-    type="fixed">
+    type="continuous">
     <origin
       xyz="0 -0.01 0"
@@ -422,5 +422,5 @@
       link="Wheel_Arm_Back_Right" />
     <axis
-      xyz="0 0 0" />
+      xyz="0 0 1" />
   </joint>
   <link
@@ -446,5 +446,5 @@
       <geometry>
         <mesh
-          filename="package://rover_urdf/meshes/Wheel_Right.STL" />
+          filename="package://rover_urdf/meshes/Wheel.STL" />
       </geometry>
       <material
@@ -465,5 +465,5 @@
     type="continuous">
     <origin
-      xyz="-0.664 -0.19693 -0.128"
+      xyz="0 0 -0.15"
       rpy="0 0 0" />
     <parent
@@ -530,5 +530,5 @@
       <origin
         xyz="0.577627534357114 0.279237097647626 0.082501913006288"
-        rpy="0 0 0" />
+        rpy="0 0 3.14" />
       <mass
         value="1.30155333808383" />
@@ -544,8 +544,8 @@
       <origin
         xyz="0 0 0"
-        rpy="0 0 0" />
-      <geometry>
-        <mesh
-          filename="package://rover_urdf/meshes/Sus_Arm_Front_Left.STL" />
+        rpy="0 0 3.14" />
+      <geometry>
+        <mesh
+          filename="package://rover_urdf/meshes/Sus_Arm_LF_RB.STL" />
       </geometry>
       <material
@@ -572,5 +572,5 @@
     type="fixed">
     <origin
-      xyz="-0.22502 -0.21159 -0.089956"
+      xyz="0.43 0.05 0"
       rpy="0 0 0" />
     <parent
@@ -603,5 +603,5 @@
       <geometry>
         <mesh
-          filename="package://rover_urdf/meshes/Wheel_Arm_Front_Left.STL" />
+          filename="package://rover_urdf/meshes/Wheel_Arm.STL" />
       </geometry>
       <material
@@ -632,5 +632,5 @@
   <joint
     name="Left_front_wheel_arm_joint"
-    type="fixed">
+    type="continuous">
     <origin
       xyz="1.7429E-05 0.003185 -4.3566E-05"
@@ -641,5 +641,5 @@
       link="Wheel_Arm_Front_Left" />
     <axis
-      xyz="0 0 0" />
+      xyz="0 0 1" />
   </joint>
   <link
@@ -665,5 +665,5 @@
       <geometry>
         <mesh
-          filename="package://rover_urdf/meshes/Wheel_Left.STL" />
+          filename="package://rover_urdf/meshes/Wheel.STL" />
       </geometry>
       <material
@@ -684,5 +684,5 @@
     type="continuous">
     <origin
-      xyz="0.664 0.19693 -0.128"
+      xyz="0 0 -0.15"
       rpy="0 0 0" />
     <parent
@@ -715,5 +715,5 @@
       <geometry>
         <mesh
-          filename="package://rover_urdf/meshes/Sus_Arm_Back_Left.STL" />
+          filename="package://rover_urdf/meshes/Sus_Arm_LB_RF.STL" />
       </geometry>
       <material
@@ -740,5 +740,5 @@
     type="fixed">
     <origin
-      xyz="0.22498 -0.23159 -0.090044"
+      xyz="-0.43 0.05 0"
       rpy="0 0 0" />
     <parent
@@ -771,5 +771,5 @@
       <geometry>
         <mesh
-          filename="package://rover_urdf/meshes/Wheel_Arm_Back_Left.STL" />
+          filename="package://rover_urdf/meshes/Wheel_Arm.STL" />
       </geometry>
       <material
@@ -800,7 +800,7 @@
   <joint
     name="Left_back_wheel_arm_joint"
-    type="fixed">
-    <origin
-      xyz="-1.328 0.012135 4.3562E-05"
+    type="continuous">
+    <origin
+      xyz="-.1 0 0"
       rpy="0 0 0" />
     <parent
@@ -809,5 +809,5 @@
       link="Wheel_Arm_Back_Left" />
     <axis
-      xyz="0 0 0" />
+      xyz="0 0 1" />
   </joint>
   <link
@@ -833,5 +833,5 @@
       <geometry>
         <mesh
-          filename="package://rover_urdf/meshes/Wheel_Left.STL" />
+          filename="package://rover_urdf/meshes/Wheel.STL" />
       </geometry>
       <material
@@ -852,5 +852,5 @@
     type="continuous">
     <origin
-      xyz="0.664 0.20693 -0.128"
+      xyz="0.0 0.0 -0.15"
       rpy="0 0 0" />
     <parent

Commit message: Fix collisions

File: src/URDF/rover_urdf/urdf/chassis_urdf.xacro (robot description, xacro)
@@ -169,5 +169,5 @@
     </visual>
     <collision>
-      <origin xyz="0.477000 -0.270000 0.084000" rpy="0.000000 0.000000 0.000000"/>
+      <origin xyz="-0.225 0.000000 0.000000" rpy="0.000000 0.000000 0.000000"/>
       <geometry>
         <box size="0.450000 0.090000 0.050000"/>
@@ -175,5 +175,5 @@
     </collision>
     <collision>
-      <origin xyz="0.624500 -0.345000 0.083000" rpy="0.000000 0.000000 0.000000"/>
+      <origin xyz="0.000000 0.000000 0.000000" rpy="0.000000 0.000000 0.000000"/>
       <geometry>
         <box size="0.085000 0.070000 0.090000"/>
@@ -225,5 +225,5 @@
     </visual>
     <collision>
-      <origin xyz="-0.664057 -0.199347 -0.131243" rpy="0.000000 0.000000 0.000000"/>
+      <origin xyz="0 0 -0.131243" rpy="0 0 0"/>
       <geometry>
         <box size="0.154965 0.097667 0.148371"/>
@@ -231,5 +231,5 @@
     </collision>
     <collision>
-      <origin xyz="-0.664057 -0.125000 -0.051243" rpy="0.000000 0.000000 0.000000"/>
+      <origin xyz="0 -0.175000 -0.051243" rpy="0 0 0"/>
       <geometry>
         <box size="0.074965 0.049667 0.228371"/>
@@ -237,5 +237,5 @@
     </collision>
     <collision>
-      <origin xyz="-0.664057 -0.219347 0.045000" rpy="0.000000 0.000000 0.000000"/>
+      <origin xyz="0 -0.08 0.045000" rpy="0 0 0"/>
       <geometry>
         <box size="0.074965 0.157667 0.068371"/>
@@ -287,5 +287,5 @@
     </visual>
     <collision>
-      <origin xyz="0.000000 -0.065254 0.000000" rpy="1.570000 0.000000 0.000000"/>
+      <origin xyz="0.000000  0.000000 0.000000" rpy="1.570000 0.000000 0.000000"/>
       <geometry>
         <cylinder radius="0.141667" length="0.139000"/>
@@ -337,5 +337,5 @@
     </visual>
     <collision>
-    <origin xyz="-0.477250 -0.271000 0.089000" rpy="0.000000 0.000000 0.000000"/>
+    <origin xyz="0.225 0 0" rpy="0.000000 0.000000 0.000000"/>
       <geometry>
         <box size="0.451125 0.077375 0.060750"/>
@@ -343,5 +343,5 @@
     </collision>
     <collision>
-      <origin xyz="-0.627250 -0.347000 0.084000" rpy="0.000000 0.000000 0.000000"/>
+      <origin xyz="0 0 0" rpy="0.000000 0.000000 0.000000"/>
       <geometry>
         <box size="0.081125 0.067375 0.090750"/>
@@ -393,5 +393,5 @@
     </visual>
     <collision>
-      <origin xyz="-0.664057 -0.199347 -0.131243" rpy="0.000000 0.000000 0.000000"/>
+      <origin xyz="0 0 -0.131243" rpy="0 0 0"/>
       <geometry>
         <box size="0.154965 0.097667 0.148371"/>
@@ -399,5 +399,5 @@
     </collision>
     <collision>
-      <origin xyz="-0.664057 -0.125000 -0.051243" rpy="0.000000 0.000000 0.000000"/>
+      <origin xyz="0 -0.175000 -0.051243" rpy="0 0 0"/>
       <geometry>
         <box size="0.074965 0.049667 0.228371"/>
@@ -405,5 +405,5 @@
     </collision>
     <collision>
-      <origin xyz="-0.664057 -0.219347 0.045000" rpy="0.000000 0.000000 0.000000"/>
+      <origin xyz="0 -0.08 0.045000" rpy="0 0 0"/>
       <geometry>
         <box size="0.074965 0.157667 0.068371"/>
@@ -455,5 +455,5 @@
     </visual>
     <collision>
-      <origin xyz="0.000000 -0.065254 0.000000" rpy="1.570000 0.000000 0.000000"/>
+      <origin xyz="0.000000 0.000000 0.000000" rpy="1.570000 0.000000 0.000000"/>
       <geometry>
         <cylinder radius="0.141667" length="0.139000"/>
@@ -556,5 +556,5 @@
     </visual>
     <collision>
-      <origin xyz="0.477000 0.270000 0.084000" rpy="0.000000 0.000000 0.000000"/>
+      <origin xyz="-0.225 0.0 0.000000" rpy="0.000000 0.000000 0.000000"/>
       <geometry>
         <box size="0.450000 0.090000 0.050000"/>
@@ -562,5 +562,5 @@
     </collision>
     <collision>
-      <origin xyz="0.624500 0.345000 0.083000" rpy="0.000000 0.000000 0.000000"/>
+      <origin xyz="0 0.000000 0.000000" rpy="0.000000 0.000000 0.000000"/>
       <geometry>
         <box size="0.085000 0.070000 0.090000"/>
@@ -612,5 +612,5 @@
     </visual>
     <collision>
-      <origin xyz="0.664057 0.199347 -0.131243" rpy="0.000000 0.000000 0.000000"/>
+      <origin xyz="0.000000 0.1 -0.131243" rpy="0.000000 0.000000 0.000000"/>
       <geometry>
         <box size="0.154965 0.097667 0.148371"/>
@@ -618,5 +618,5 @@
     </collision>
     <collision>
-      <origin xyz="0.664057 0.125000 -0.051243" rpy="0.000000 0.000000 0.000000"/>
+      <origin xyz="0.000000 0.14 -0.051243" rpy="0.000000 0.000000 0.000000"/>
       <geometry>
         <box size="0.074965 0.049667 0.228371"/>
@@ -624,5 +624,5 @@
     </collision>
     <collision>
-      <origin xyz="0.664057 0.219347 0.045000" rpy="0.000000 0.000000 0.000000"/>
+      <origin xyz="0.000000 0.05 0.045000" rpy="0.000000 0.000000 0.000000"/>
       <geometry>
         <box size="0.074965 0.157667 0.068371"/>
@@ -674,5 +674,5 @@
     </visual>
     <collision>
-      <origin xyz="0.000000 0.065254 0.000000" rpy="1.570000 0.000000 0.000000"/>
+      <origin xyz="0.000000 0.000000 0.000000" rpy="1.570000 0.000000 0.000000"/>
       <geometry>
         <cylinder radius="0.141667" length="0.139000"/>
@@ -724,5 +724,5 @@
     </visual>
     <collision>
-    <origin xyz="-0.477250 0.271000 0.089000" rpy="0.000000 0.000000 0.000000"/>
+    <origin xyz="0.225 0.000000 0.000000" rpy="0.000000 0.000000 0.000000"/>
       <geometry>
         <box size="0.451125 0.077375 0.060750"/>
@@ -730,5 +730,5 @@
     </collision>
     <collision>
-      <origin xyz="-0.627250 0.347000 0.084000" rpy="0.000000 0.000000 0.000000"/>
+      <origin xyz="0.0 0.000000 0.000000" rpy="0.000000 0.000000 0.000000"/>
       <geometry>
         <box size="0.081125 0.067375 0.090750"/>
@@ -780,5 +780,5 @@
     </visual>
     <collision>
-      <origin xyz="0.664057 0.199347 -0.131243" rpy="0.000000 0.000000 0.000000"/>
+      <origin xyz="0.000000 0.1 -0.131243" rpy="0.000000 0.000000 0.000000"/>
       <geometry>
         <box size="0.154965 0.097667 0.148371"/>
@@ -786,5 +786,5 @@
     </collision>
     <collision>
-      <origin xyz="0.664057 0.125000 -0.051243" rpy="0.000000 0.000000 0.000000"/>
+      <origin xyz="0.000000 0.14 -0.051243" rpy="0.000000 0.000000 0.000000"/>
       <geometry>
         <box size="0.074965 0.049667 0.228371"/>
@@ -792,5 +792,5 @@
     </collision>
     <collision>
-      <origin xyz="0.664057 0.219347 0.045000" rpy="0.000000 0.000000 0.000000"/>
+      <origin xyz="0.000000 0.05 0.045000" rpy="0.000000 0.000000 0.000000"/>
       <geometry>
         <box size="0.074965 0.157667 0.068371"/>
@@ -842,5 +842,5 @@
     </visual>
     <collision>
-      <origin xyz="0.000000 0.065254 0.000000" rpy="1.570000 0.000000 0.000000"/>
+      <origin xyz="0.000000 0.000000 0.000000" rpy="1.570000 0.000000 0.000000"/>
       <geometry>
         <cylinder radius="0.141667" length="0.139000"/>
